File: Electronics/Mainboard/DAC.sch (KiCad schematic (older format))
At the start: 28 parts, among them U1 OPA2277, U2 OPA2277

Commit message: Many changes. I lost track of them...
Parts:
- removed U1: OPA2277, Package_SO:SOIC-8_3.9x4.9mm_P1.27mm, symbol Amplifier_Operational:OPA2277
- removed U2: OPA2277, symbol Amplifier_Operational:OPA2277
- added U1, U2: AD8676, Package_SO:SOIC-8_3.9x4.9mm_P1.27mm, symbol STM_Custom_Lib:AD8676
- C1, C2, C3, C4: value 4u7 -> 10u; footprint (none) -> Capacitor_SMD:C_1206_3216Metric_Pad1.42x1.75mm_HandSolder
- C5, C6, C7, C8, R1, R10, R11, R12, R13, R14, R15, R16, R17, R18, R2, R3, R4, R5, R6, R7, R8, R9: footprint (none) -> Capacitor_SMD:C_0805_2012Metric_Pad1.15x1.40mm_HandSolder
Connections:
- net +15V: now also C2.1, C6.1, U1.8 (V+), U2.8 (V+); no longer C1.1, C5.1
- net -15V: now also C1.2, C5.2, U1.4 (V-), U2.4 (V-); no longer C2.2, C6.2
- net GND: now also C1.1, C2.2, C5.1, C6.2; no longer C1.2, C2.1, C5.2, C6.1, R10.1, R9.1
- net at R14.1, R18.2: now also U2.7
- net at R14.2, R7.1: now also U2.5 (+)
- net at R13.1, R17.2: now also U2.1
- net at R13.2, R5.1, R6.1: now also U2.3 (+)
- net at R8.1: now also R10.1, U2.6 (-); no longer R10.2
- net at R12.1, R16.2: now also U1.7
- net at R12.2, R3.1: now also U1.5 (+)
- net at R11.1, R15.2: now also U1.1
- net at R1.1, R11.2, R2.1: now also U1.3 (+)
- net at R4.1: now also R9.1, U1.6 (-); no longer R9.2
- new net GNDA: R10.2, R9.2, U1.2 (-), U2.2 (-)
Other:
- moved on the sheet: C3, C7, R13, R18
