File: Electronics/Mainboard/Mainboard.kicad_pcb (KiCad board)
At the start: 2 copper layers, 160 x 120 mm, 129 parts, among them J1 Conn_Coaxial, J2 DB25_Male_MountingHoles, J3 609-5192-ND, J4 609-5192-ND, J7 Conn_Coaxial, U1 AD8676, U10 AD8675, U11 AD5781, U12 AD8676xR, U13 AD8675, U14 LM75C, U15 Beaglebone_Black, U2 AD8676, U3 LT1469, U4 LTC2326-16, U5 AD5781, U6 AD8676xR, U7 AD8675, U8 AD5781, U9 AD8676xR

Commit message: Layout of piezo DACs ready
Parts:
- added C100: 10u, Capacitor_SMD:C_0805_2012Metric_Pad1.15x1.40mm_HandSolder, F.Cu at (237.3, 37.6)
- added C101: 10u, Capacitor_SMD:C_0805_2012Metric_Pad1.15x1.40mm_HandSolder, F.Cu at (250.4, 29.6)
- added C102: 10u, Capacitor_SMD:C_0805_2012Metric_Pad1.15x1.40mm_HandSolder, F.Cu at (250.4, 32.5)
- added C103: 100n, Capacitor_SMD:C_0603_1608Metric_Pad1.05x0.95mm_HandSolder, F.Cu at (263.8, 22.9)
- added C104: 100n, Capacitor_SMD:C_0603_1608Metric_Pad1.05x0.95mm_HandSolder, F.Cu at (251.0, 37.8)
- added C105: 100n, Capacitor_SMD:C_0603_1608Metric_Pad1.05x0.95mm_HandSolder, F.Cu at (255.0, 33.8)
- added C83: opt, Capacitor_SMD:C_0603_1608Metric_Pad1.05x0.95mm_HandSolder, F.Cu at (202.7, 49.6)
- added C84: opt, Capacitor_SMD:C_0603_1608Metric_Pad1.05x0.95mm_HandSolder, F.Cu at (201.3, 63.3)
- added C85: opt, Capacitor_SMD:C_0603_1608Metric_Pad1.05x0.95mm_HandSolder, F.Cu at (202.7, 70.4)
- added C86: opt, Capacitor_SMD:C_0603_1608Metric_Pad1.05x0.95mm_HandSolder, F.Cu at (201.3, 84.1)
- added C87: opt, Capacitor_SMD:C_0603_1608Metric_Pad1.05x0.95mm_HandSolder, F.Cu at (191.6, 59.4)
- added C88: opt, Capacitor_SMD:C_0603_1608Metric_Pad1.05x0.95mm_HandSolder, F.Cu at (191.6, 80.2)
- added C89: 10p, Capacitor_SMD:C_0603_1608Metric_Pad1.05x0.95mm_HandSolder, F.Cu at (255.0, 28.8)
- added C90: 10p, Capacitor_SMD:C_0603_1608Metric_Pad1.05x0.95mm_HandSolder, F.Cu at (263.4, 25.9)
- added C91: 10p, Capacitor_SMD:C_0603_1608Metric_Pad1.05x0.95mm_HandSolder, F.Cu at (259.3, 28.4)
- added C92: 10u, Capacitor_SMD:C_0805_2012Metric_Pad1.15x1.40mm_HandSolder, F.Cu at (254.5, 23.1)
- added C93: 10u, Capacitor_SMD:C_0805_2012Metric_Pad1.15x1.40mm_HandSolder, F.Cu at (242.1, 38.4)
- added C94: 100n, Capacitor_SMD:C_0603_1608Metric_Pad1.05x0.95mm_HandSolder, F.Cu at (250.2, 35.3)
- added C95: 100n, Capacitor_SMD:C_0603_1608Metric_Pad1.05x0.95mm_HandSolder, F.Cu at (255.0, 31.3)
- added C96: 10u, Capacitor_SMD:C_0805_2012Metric_Pad1.15x1.40mm_HandSolder, F.Cu at (259.3, 23.1)
- added C97: 10u, Capacitor_SMD:C_0805_2012Metric_Pad1.15x1.40mm_HandSolder, F.Cu at (254.5, 26.1)
- added C98: 100n, Capacitor_SMD:C_0603_1608Metric_Pad1.05x0.95mm_HandSolder, F.Cu at (259.1, 25.9)
- added C99: 100n, Capacitor_SMD:C_0603_1608Metric_Pad1.05x0.95mm_HandSolder, F.Cu at (246.6, 38.2)
- added JP10: Jumper, Connector_PinHeader_2.54mm:PinHeader_1x02_P2.54mm_Vertical, F.Cu at (245.7, 32.0)
- added JP3: Jumper, Connector_PinHeader_2.54mm:PinHeader_1x02_P2.54mm_Vertical, F.Cu at (189.7, 76.0)
- added JP4: Jumper, Connector_PinHeader_2.54mm:PinHeader_1x02_P2.54mm_Vertical, F.Cu at (189.7, 96.8)
- added JP5: Jumper, Connector_PinHeader_2.54mm:PinHeader_1x02_P2.54mm_Vertical, F.Cu at (189.7, 55.1)
- added JP6: Jumper, Connector_PinHeader_2.54mm:PinHeader_1x02_P2.54mm_Vertical, F.Cu at (210.8, 53.9)
- added JP7: Jumper, Connector_PinHeader_2.54mm:PinHeader_1x02_P2.54mm_Vertical, F.Cu at (210.8, 61.3)
- added JP8: Jumper, Connector_PinHeader_2.54mm:PinHeader_1x02_P2.54mm_Vertical, F.Cu at (210.8, 74.7)
- added JP9: Jumper, Connector_PinHeader_2.54mm:PinHeader_1x02_P2.54mm_Vertical, F.Cu at (210.8, 82.1)
- added U16: AD5781, Package_SO:TSSOP-20_4.4x6.5mm_P0.65mm, F.Cu at (239.3, 25.7)
- added U17: AD8676xR, Package_SO:SOIC-8_3.9x4.9mm_P1.27mm, F.Cu at (247.9, 24.9)
- added U18: AD8675, Package_SO:SOIC-8_3.9x4.9mm_P1.27mm, F.Cu at (239.2, 32.9)
- C1, C2, C3, C4: value 10u -> 100n; footprint Capacitor_SMD:C_1206_3216Metric_Pad1.42x1.75mm_HandSolder -> Capacitor_SMD:C_0603_1608Metric_Pad1.05x0.95mm_HandSolder
- C26, C30: value 10p -> 100n
- C27, C29, C31, C37, C41, C45, C46, C48, C52, C57, C60, C63, C68: footprint Capacitor_SMD:C_0805_2012Metric_Pad1.15x1.40mm_HandSolder -> Capacitor_SMD:C_0603_1608Metric_Pad1.05x0.95mm_HandSolder
- C32, C36, C40, C64, C69, C70: value 10u -> 100n; footprint Capacitor_SMD:C_0805_2012Metric_Pad1.15x1.40mm_HandSolder -> Capacitor_SMD:C_0603_1608Metric_Pad1.05x0.95mm_HandSolder
- C33, C71, C72, C75, C76: value 100n -> 10p; footprint Capacitor_SMD:C_0805_2012Metric_Pad1.15x1.40mm_HandSolder -> Capacitor_SMD:C_0603_1608Metric_Pad1.05x0.95mm_HandSolder
- C38, C42, C5, C53, C56, C6, C61, C67, C7, C8: value 100n -> 10u
- C49, C73, C74: value 10u -> 10p; footprint Capacitor_SMD:C_0805_2012Metric_Pad1.15x1.40mm_HandSolder -> Capacitor_SMD:C_0603_1608Metric_Pad1.05x0.95mm_HandSolder
- moved N1 281.3 mm to (-124.6, 161.4), turned to 0 degrees
- moved C75 147.5 mm to (165.6, 91.9), turned to 180 degrees
- moved C76 147.4 mm to (163.7, 101.0), turned to 180 degrees
- moved C73 142.4 mm to (165.6, 71.1), turned to 180 degrees
- moved C62 138.6 mm to (161.7, 73.7), turned to 90 degrees
- moved C70 137.4 mm to (171.1, 69.5), turned to 90 degrees
- moved C72 136.1 mm to (163.7, 59.4), turned to 180 degrees
- moved C74 135.5 mm to (163.7, 80.2), turned to 180 degrees
- moved C64 129.4 mm to (163.7, 73.7), turned to 90 degrees
- moved C63 129.1 mm to (168.2, 80.2), turned to 180 degrees
- moved C69 127.1 mm to (178.6, 76.6), turned to 270 degrees
- moved C66 126.0 mm to (181.2, 77.6), turned to 180 degrees
- moved C71 124.8 mm to (165.6, 50.3), turned to 180 degrees
- moved C67 122.3 mm to (169.2, 69.5), turned to 90 degrees
- moved U12 119.3 mm to (167.2, 75.6), turned to 270 degrees
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Connections:
- net /DAC/sheet5DAA3250/!SYNC renamed /Piezo-DACs/~CS-Y
- net /DAC/sheet5DAA6516/!SYNC renamed /Piezo-DACs/~CS-X
- net /DAC/sheet5DAB2C4D/!SYNC renamed /Piezo-DACs/~CS-Z
- C1 pad 1: GND -> /+20V
- C1 pad 2: -15V -> GND
- C2 pad 1: +15V -> GND
- C2 pad 2: GND -> /-20V
- C26 pad 1: /DAC/Z -> GND
- C26 pad 2: Net-(C26-Pad2) -> -15V
- C27 pad 1: +3V3 -> +15V
- C27 pad 2: GNDD -> GND
- C28 pad 1: /DAC/X -> Net-(C28-Pad1)
- C29 pad 1: +3V3 -> GND
- C29 pad 2: GNDD -> -15V
- C3 pad 1: +15V -> /+20V
- C30 pad 1: /DAC/Y -> +15V
- C30 pad 2: Net-(C30-Pad2) -> GND
- C31 pad 1: +3V3 -> GND
- C31 pad 2: GNDD -> -15V
- C32 pad 1: +3V3 -> /3V3
- C32 pad 2: GNDD -> GND
- C33 pad 1: +3V3 -> Net-(C33-Pad1)
- C33 pad 2: GNDD -> Net-(C33-Pad2)
- C34 pad 1: +3V3 -> +15V
- C34 pad 2: GNDD -> GND
- C35 pad 1: +15V -> GND
- C35 pad 2: GNDA -> -15V
- C36 pad 1: GNDA -> +15V
- C36 pad 2: -15V -> GND
- C37 pad 1: +15V -> GND
- C37 pad 2: GNDA -> -15V
- C38 pad 1: GNDA -> +15V
- C38 pad 2: -15V -> GND
- C39 pad 1: +15V -> GND
- C39 pad 2: GNDA -> -15V
- C4 pad 2: -15V -> /-20V
- C40 pad 1: GNDA -> +15V
- C40 pad 2: -15V -> GND
- C41 pad 1: +15V -> GND
- C41 pad 2: GNDA -> -15V
- C42 pad 1: GNDA -> +15V
- C42 pad 2: -15V -> GND
- C43 pad 1: +15V -> GND
- C43 pad 2: GNDA -> -15V
- C44 pad 1: GNDA -> /3V3
- C44 pad 2: -15V -> GND
- C45 pad 2: GNDA -> GND
- C46 pad 1: GNDA -> GND
- C47 pad 1: +3V3 -> /3V3
- C47 pad 2: GNDD -> GND
- C48 pad 1: +3V3 -> /3V3
- C48 pad 2: GNDD -> GND
- C49 pad 1: +3V3 -> Net-(C49-Pad1)
- C49 pad 2: GNDD -> Net-(C49-Pad2)
- C5 pad 1: GND -> /+20V
- C5 pad 2: -15V -> GND
- C50 pad 2: GNDA -> GND
- C51 pad 1: GNDA -> GND
- C52 pad 2: GNDA -> GND
- C53 pad 1: GNDA -> +15V
- C53 pad 2: -15V -> GND
- C54 pad 2: GNDA -> GND
- C55 pad 1: GNDA -> GND
- C56 pad 1: +15V -> GND
- C56 pad 2: GNDA -> -15V
- C57 pad 1: GNDA -> +15V
- C57 pad 2: -15V -> GND
- C58 pad 2: GNDA -> GND
- C59 pad 1: GNDA -> GND
- C6 pad 1: +15V -> GND
- C6 pad 2: GND -> /-20V
- C60 pad 1: +15V -> GND
- C60 pad 2: GNDA -> -15V
- C61 pad 1: GNDA -> +15V
- C61 pad 2: -15V -> GND
- C62 pad 1: +3V3 -> GND
- C62 pad 2: GNDD -> -15V
- C63 pad 1: +3V3 -> +15V
- C63 pad 2: GNDD -> GND
- C64 pad 1: +3V3 -> GND
- C64 pad 2: GNDD -> -15V
- C65 pad 2: GNDA -> GND
- C66 pad 1: GNDA -> GND
- C67 pad 1: +15V -> /3V3
- C67 pad 2: GNDA -> GND
- C68 pad 1: GNDA -> +15V
- C68 pad 2: -15V -> GND
- C69 pad 1: +15V -> GND
- C69 pad 2: GNDA -> -15V
- C7 pad 1: +15V -> /+20V
- C70 pad 1: GNDA -> /3V3
- C70 pad 2: -15V -> GND
- C71 pad 1: +15V -> /Piezo-DACs/REF_P
- C71 pad 2: GNDA -> GND
- C72 pad 1: GNDA -> /Piezo-DACs/REF_N
- C72 pad 2: -15V -> GND
- C73 pad 1: +15V -> /Piezo-DACs/REF_P
- C73 pad 2: GNDA -> GND
- C74 pad 1: GNDA -> /Piezo-DACs/REF_N
- C74 pad 2: -15V -> GND
- C75 pad 1: +15V -> /Piezo-DACs/REF_P
- C75 pad 2: GNDA -> GND
- C76 pad 1: GNDA -> /Piezo-DACs/REF_N
- C76 pad 2: -15V -> GND
- C77 pad 1: /Power/analog_-15V -> -15V
- C77 pad 2: /Power/analog_gnd -> GND
- C78 pad 1: /Power/analog_gnd -> GND
- C78 pad 2: /Power/analog_+15V -> +15V
- C79 pad 1: /Power/piezo_-20V -> /-20V
- C79 pad 2: /Power/piezo_gnd -> GND
- C8 pad 2: -15V -> /-20V
- C80 pad 1: /Power/piezo_gnd -> GND
- C80 pad 2: /Power/piezo_+20V -> /+20V
- C81 pad 1: /Power/digital_3V3 -> /3V3
- C81 pad 2: /Beaglebone/GND -> GND
- C82 pad 1: /Beaglebone/GND -> GND
- J2 pad 1: /Power/analog_-15V -> -15V
- J2 pad 14: /Power/analog_-15V -> -15V
- J2 pad 15: /Power/analog_gnd -> GND
- J2 pad 16: /Power/analog_+15V -> +15V
- J2 pad 17: /Power/piezo_-20V -> /-20V
- J2 pad 18: /Power/piezo_gnd -> GND
- J2 pad 19: /Power/piezo_+20V -> /+20V
- J2 pad 2: /Power/analog_gnd -> GND
- J2 pad 20: /Power/digital_3V3 -> /3V3
- J2 pad 21: /Beaglebone/GND -> GND
- J2 pad 3: /Power/analog_+15V -> +15V
- J2 pad 4: /Power/piezo_-20V -> /-20V
- J2 pad 5: /Power/piezo_gnd -> GND
- J2 pad 6: /Power/piezo_+20V -> /+20V
- J2 pad 7: /Power/digital_3V3 -> /3V3
- J2 pad 8: /Beaglebone/GND -> GND
- J3 pad 6: Net-(J3-Pad6) -> /Piezo-DACs/Z+X
- J3 pad 7: Net-(J3-Pad7) -> /Piezo-DACs/Z-X
- J3 pad 8: Net-(J3-Pad8) -> /Piezo-DACs/Z+Y
- J3 pad 9: Net-(J3-Pad9) -> /Piezo-DACs/Z-Y
- R1 pad 2: /DAC/Z -> /Piezo-DACs/Z
- R10 pad 2: GNDA -> GND
- R15 pad 1: /DAC/Z+X -> Net-(JP6-Pad1)
- R16 pad 1: /DAC/Z-X -> Net-(JP7-Pad1)
- R17 pad 1: /DAC/Z+Y -> Net-(JP8-Pad1)
- R18 pad 1: /DAC/Z-Y -> Net-(JP9-Pad1)
- R2 pad 2: /DAC/X -> /Piezo-DACs/X
- R3 pad 2: /DAC/Z -> /Piezo-DACs/Z
- R4 pad 2: /DAC/X -> /Piezo-DACs/X
- R5 pad 2: /DAC/Z -> /Piezo-DACs/Z
- R6 pad 2: /DAC/Y -> /Piezo-DACs/Y
- R7 pad 2: /DAC/Z -> /Piezo-DACs/Y
- R8 pad 2: /DAC/Y -> /Piezo-DACs/Z
- R9 pad 2: GNDA -> GND
- U1 pad 2: GNDA -> GND
- U1 pad 4: -15V -> /-20V
- U1 pad 8: +15V -> /+20V
- U10 pad 6: /DAC/X -> Net-(C28-Pad1)
- U11 pad 1: Net-(C30-Pad2) -> Net-(C49-Pad2)
- U11 pad 10: +3V3 -> /3V3
- U11 pad 11: /DAC/sheet5DAB2C4D/SDO -> /Piezo-DACs/MISO
- U11 pad 12: /DAC/sheet5DAB2C4D/SDIN -> /Piezo-DACs/MOSI
- U11 pad 13: /DAC/sheet5DAB2C4D/SCLK -> /Piezo-DACs/CLK
- U11 pad 15: GNDD -> GND
- U11 pad 19: GNDA -> GND
- U11 pad 20: /DAC/Y -> Net-(C49-Pad1)
- U11 pad 6: /DAC/sheet5DAB2C4D/!RST -> /3V3
- U11 pad 7: /DAC/sheet5DAB2C4D/!CLR -> /3V3
- U11 pad 8: /DAC/sheet5DAB2C4D/!LDAC -> /Piezo-DACs/~LDAC
- U11 pad 9: +3V3 -> /3V3
- U12 pad 3: /DAC/REF_P -> /Piezo-DACs/REF_P
- U12 pad 5: /DAC/REF_N -> /Piezo-DACs/REF_N
- U13 pad 2: Net-(C30-Pad2) -> Net-(C49-Pad2)
- U13 pad 6: /DAC/Y -> Net-(C49-Pad1)
- U15 pad P8_1: /Beaglebone/GND -> GND
- U15 pad P8_2: /Beaglebone/GND -> GND
- U15 pad P9_1: /Beaglebone/GND -> GND
- U15 pad P9_2: /Beaglebone/GND -> GND
- U15 pad P9_43: /Beaglebone/GND -> GND
- U15 pad P9_44: /Beaglebone/GND -> GND
- U15 pad P9_45: /Beaglebone/GND -> GND
- U15 pad P9_46: /Beaglebone/GND -> GND
- U2 pad 2: GNDA -> GND
- U2 pad 4: -15V -> /-20V
- U2 pad 8: +15V -> /+20V
- U5 pad 1: Net-(C26-Pad2) -> Net-(C33-Pad2)
- U5 pad 10: +3V3 -> /3V3
- U5 pad 11: /DAC/sheet5DAA3250/SDO -> /Piezo-DACs/MISO
- U5 pad 12: /DAC/sheet5DAA3250/SDIN -> /Piezo-DACs/MOSI
- U5 pad 13: /DAC/sheet5DAA3250/SCLK -> /Piezo-DACs/CLK
- U5 pad 15: GNDD -> GND
- U5 pad 19: GNDA -> GND
- U5 pad 20: /DAC/Z -> Net-(C33-Pad1)
- U5 pad 6: /DAC/sheet5DAA3250/!RST -> /3V3
- U5 pad 7: /DAC/sheet5DAA3250/!CLR -> /3V3
- U5 pad 8: /DAC/sheet5DAA3250/!LDAC -> /Piezo-DACs/~LDAC
- U5 pad 9: +3V3 -> /3V3
- U6 pad 3: /DAC/REF_P -> /Piezo-DACs/REF_P
- U6 pad 5: /DAC/REF_N -> /Piezo-DACs/REF_N
- U7 pad 2: Net-(C26-Pad2) -> Net-(C33-Pad2)
- U7 pad 6: /DAC/Z -> Net-(C33-Pad1)
- U8 pad 10: +3V3 -> /3V3
- U8 pad 11: /DAC/sheet5DAA6516/SDO -> /Piezo-DACs/MISO
- U8 pad 12: /DAC/sheet5DAA6516/SDIN -> /Piezo-DACs/MOSI
- U8 pad 13: /DAC/sheet5DAA6516/SCLK -> /Piezo-DACs/CLK
- U8 pad 15: GNDD -> GND
- U8 pad 19: GNDA -> GND
- U8 pad 20: /DAC/X -> Net-(C28-Pad1)
- U8 pad 6: /DAC/sheet5DAA6516/!RST -> /3V3
- U8 pad 7: /DAC/sheet5DAA6516/!CLR -> /3V3
- U8 pad 8: /DAC/sheet5DAA6516/!LDAC -> /Piezo-DACs/~LDAC
- U8 pad 9: +3V3 -> /3V3
- U9 pad 3: /DAC/REF_P -> /Piezo-DACs/REF_P
- U9 pad 5: /DAC/REF_N -> /Piezo-DACs/REF_N
Routing:
- net GND: track 0.00 -> 76.5 mm, vias 0 -> 70
- net /Piezo-DACs/REF_P: track 0.00 -> 76.3 mm, vias 0 -> 3
- net /Piezo-DACs/REF_N: track 0.00 -> 75.9 mm, vias 0 -> 3
- net /Piezo-DACs/CLK: track 0.00 -> 71.1 mm, vias 0 -> 3
- net /Piezo-DACs/~LDAC: track 0.00 -> 68.9 mm, vias 0 -> 3
- net /Piezo-DACs/MOSI: track 0.00 -> 68.9 mm, vias 0 -> 3
- net /3V3: track 0.00 -> 68.8 mm
- net /Piezo-DACs/MISO: track 0.00 -> 67.1 mm, vias 0 -> 3
- net +15V: track 0.00 -> 51.5 mm, vias 0 -> 27
- net -15V: track 0.00 -> 46.4 mm, vias 0 -> 15
- net Net-(C49-Pad1): track 0.00 -> 22.7 mm
- net Net-(C28-Pad1): track 0.00 -> 22.7 mm
- net Net-(C33-Pad1): track 0.00 -> 22.7 mm
- net /Piezo-DACs/Z: track 0.00 -> 22.0 mm, vias 0 -> 2
- net /Piezo-DACs/Y: track 0.00 -> 19.6 mm, vias 0 -> 2
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- added copper zone on B.Cu, net +15V
- added copper zone on F.Cu, net +15V
- added copper zone on B.Cu, net -15V
- added copper zone on F.Cu, net -15V
- added copper zone on B.Cu, net /+20V
- added copper zone on B.Cu, net /-20V
- added copper zone on B.Cu, net GND
- added copper zone on F.Cu, net GND
Other:
- net class Default: trace_width 0.25 -> 0.2

Commit message: ADC Schematic
Parts:
- C10, C9: value 100n -> 66n; footprint Capacitor_SMD:C_0805_2012Metric_Pad1.15x1.40mm_HandSolder -> Capacitor_SMD:C_0603_1608Metric_Pad1.05x0.95mm_HandSolder
- C11, C12, C20, C23, C25: footprint Capacitor_SMD:C_1206_3216Metric_Pad1.42x1.75mm_HandSolder -> Capacitor_SMD:C_0805_2012Metric_Pad1.15x1.40mm_HandSolder
- C13, C14: value 66n -> 100n; footprint Capacitor_SMD:C_0805_2012Metric_Pad1.15x1.40mm_HandSolder -> Capacitor_SMD:C_0603_1608Metric_Pad1.05x0.95mm_HandSolder
- C15, C16, C17, C19, C21, C22, C24: footprint Capacitor_SMD:C_0805_2012Metric_Pad1.15x1.40mm_HandSolder -> Capacitor_SMD:C_0603_1608Metric_Pad1.05x0.95mm_HandSolder
- JP1, JP2: value SolderJumper_2_Bridged -> Jumper; footprint Jumper:SolderJumper-2_P1.3mm_Bridged_RoundedPad1.0x1.5mm -> Connector_PinHeader_2.54mm:PinHeader_1x02_P2.54mm_Vertical
- U4: value LTC2326-16 -> LTC2338-18
- moved C90 138.4 mm to (163.7, 121.8), turned to 180 degrees
- moved C96 135.7 mm to (168.2, 123.7), turned to 180 degrees
- moved C98 132.1 mm to (168.2, 121.8), turned to 180 degrees
- moved C97 128.7 mm to (161.7, 115.3), turned to 90 degrees
- moved U17 122.6 mm to (167.2, 117.2), turned to 270 degrees
- moved C89 122.6 mm to (165.6, 112.7), turned to 180 degrees
- moved C95 121.5 mm to (175.7, 123.4), turned to 90 degrees
- moved C103 118.4 mm to (189.0, 114.6)
- moved C92 117.2 mm to (177.0, 111.0), turned to 90 degrees
- moved C105 114.0 mm to (171.1, 111.0), turned to 90 degrees
- moved C99 113.3 mm to (163.7, 115.3), turned to 90 degrees
- moved C101 113.2 mm to (181.2, 119.2), turned to 180 degrees
- moved C102 113.0 mm to (169.2, 111.0), turned to 90 degrees
- moved C91 112.9 mm to (183.2, 111.7), turned to 180 degrees
- moved U16 112.4 mm to (174.1, 117.2), turned to 270 degrees
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Connections:
- net +5VA renamed /ADC/+5V
- net /Bias-DAC/OUT renamed /Bias
- net /Bias-DAC/~CS renamed /~CS-Bias
- net /Piezo-DACs/~CS-X renamed /~CS-X
- net /Piezo-DACs/~CS-Y renamed /~CS-Y
- net /Piezo-DACs/~CS-Z renamed /~CS-Z
- net Net-(R19-Pad2) renamed /ADC/IN+
- net Net-(R20-Pad2) renamed /ADC/IN-
- C1 pad 2: GND -> /GND
- C10 pad 2: -15V -> /GND
- C100 pad 1: /Bias-DAC/+15V -> /+15V
- C100 pad 2: /Bias-DAC/GND -> /GND
- C101 pad 1: /Bias-DAC/GND -> /GND
- C101 pad 2: /Bias-DAC/-15V -> /-15V
- C102 pad 1: /Bias-DAC/3V3 -> /3V3
- C102 pad 2: /Bias-DAC/GND -> /GND
- C103 pad 1: /Bias-DAC/+15V -> /+15V
- C103 pad 2: /Bias-DAC/GND -> /GND
- C104 pad 1: /Bias-DAC/GND -> /GND
- C104 pad 2: /Bias-DAC/-15V -> /-15V
- C105 pad 1: /Bias-DAC/3V3 -> /3V3
- C105 pad 2: /Bias-DAC/GND -> /GND
- C11 pad 1: +15V -> /+15V
- C11 pad 2: Net-(C10-Pad1) -> /GND
- C12 pad 1: Net-(C10-Pad1) -> /GND
- C12 pad 2: -15V -> /-15V
- C13 pad 1: Net-(C13-Pad1) -> /+15V
- C13 pad 2: GND -> /GND
- C14 pad 1: Net-(C14-Pad1) -> /GND
- C14 pad 2: GND -> /-15V
- C15 pad 2: GND -> /GND
- C16 pad 2: GND -> /GND
- C18 pad 2: GND -> /GND
- C19 pad 2: GND -> /GND
- C2 pad 1: GND -> /GND
- C20 pad 1: GND -> Net-(C20-Pad1)
- C20 pad 2: Net-(C20-Pad2) -> /GND
- C21 pad 1: GND -> Net-(C20-Pad1)
- C21 pad 2: Net-(C20-Pad2) -> /GND
- C22 pad 2: GND -> /GND
- C23 pad 2: GND -> /GND
- C24 pad 1: +3V3 -> /3V3
- C24 pad 2: GND -> /GND
- C25 pad 1: +3V3 -> /3V3
- C25 pad 2: GND -> /GND
- C26 pad 1: GND -> /GND
- C26 pad 2: -15V -> /-15V
- C27 pad 1: +15V -> /+15V
- C27 pad 2: GND -> /GND
- C29 pad 1: GND -> /GND
- C29 pad 2: -15V -> /-15V
- C3 pad 2: GND -> /GND
- C30 pad 1: +15V -> /+15V
- C30 pad 2: GND -> /GND
- C31 pad 1: GND -> /GND
- C31 pad 2: -15V -> /-15V
- C32 pad 2: GND -> /GND
- C34 pad 1: +15V -> /+15V
- C34 pad 2: GND -> /GND
- C35 pad 1: GND -> /GND
- C35 pad 2: -15V -> /-15V
- C36 pad 1: +15V -> /+15V
- C36 pad 2: GND -> /GND
- C37 pad 1: GND -> /GND
- C37 pad 2: -15V -> /-15V
- C38 pad 1: +15V -> /+15V
- C38 pad 2: GND -> /GND
- C39 pad 1: GND -> /GND
- C39 pad 2: -15V -> /-15V
- C4 pad 1: GND -> /GND
- C40 pad 1: +15V -> /+15V
- C40 pad 2: GND -> /GND
- C41 pad 1: GND -> /GND
- C41 pad 2: -15V -> /-15V
- C42 pad 1: +15V -> /+15V
- C42 pad 2: GND -> /GND
- C43 pad 1: GND -> /GND
- C43 pad 2: -15V -> /-15V
- C44 pad 2: GND -> /GND
- C45 pad 1: +15V -> /+15V
- C45 pad 2: GND -> /GND
- C46 pad 1: GND -> /GND
- C46 pad 2: -15V -> /-15V
- C47 pad 2: GND -> /GND
- C48 pad 2: GND -> /GND
- C5 pad 2: GND -> /GND
- C50 pad 1: +15V -> /+15V
- C50 pad 2: GND -> /GND
- C51 pad 1: GND -> /GND
- C51 pad 2: -15V -> /-15V
- C52 pad 1: +15V -> /+15V
- C52 pad 2: GND -> /GND
- C53 pad 1: +15V -> /+15V
- C53 pad 2: GND -> /GND
- C54 pad 1: +15V -> /+15V
- C54 pad 2: GND -> /GND
- C55 pad 1: GND -> /GND
- C55 pad 2: -15V -> /-15V
- C56 pad 1: GND -> /GND
- C56 pad 2: -15V -> /-15V
- C57 pad 1: +15V -> /+15V
- C57 pad 2: GND -> /GND
- C58 pad 1: +15V -> /+15V
- C58 pad 2: GND -> /GND
- C59 pad 1: GND -> /GND
- C59 pad 2: -15V -> /-15V
- C6 pad 1: GND -> /GND
- C60 pad 1: GND -> /GND
- C60 pad 2: -15V -> /-15V
- C61 pad 1: +15V -> /+15V
- C61 pad 2: GND -> /GND
- C62 pad 1: GND -> /GND
- C62 pad 2: -15V -> /-15V
- C63 pad 1: +15V -> /+15V
- C63 pad 2: GND -> /GND
- C64 pad 1: GND -> /GND
- C64 pad 2: -15V -> /-15V
- C65 pad 1: +15V -> /+15V
- C65 pad 2: GND -> /GND
- C66 pad 1: GND -> /GND
- C66 pad 2: -15V -> /-15V
- C67 pad 2: GND -> /GND
- C68 pad 1: +15V -> /+15V
- C68 pad 2: GND -> /GND
- C69 pad 1: GND -> /GND
- C69 pad 2: -15V -> /-15V
- C7 pad 2: GND -> /GND
- C70 pad 2: GND -> /GND
- C71 pad 1: /Piezo-DACs/REF_P -> /REF_P
- C71 pad 2: GND -> /GND
- C72 pad 1: /Piezo-DACs/REF_N -> /REF_N
- C72 pad 2: GND -> /GND
- C73 pad 1: /Piezo-DACs/REF_P -> /REF_P
- C73 pad 2: GND -> /GND
- C74 pad 1: /Piezo-DACs/REF_N -> /REF_N
- C74 pad 2: GND -> /GND
- C75 pad 1: /Piezo-DACs/REF_P -> /REF_P
- C75 pad 2: GND -> /GND
- C76 pad 1: /Piezo-DACs/REF_N -> /REF_N
- C76 pad 2: GND -> /GND
- C77 pad 1: -15V -> /-15V
- C77 pad 2: GND -> /GND
- C78 pad 1: GND -> /GND
- C78 pad 2: +15V -> /+15V
- C79 pad 2: GND -> /GND
- C8 pad 1: GND -> /GND
- C80 pad 1: GND -> /GND
- C81 pad 2: GND -> /GND
- C82 pad 1: GND -> /GND
- C87 pad 1: GND -> /GND
- C88 pad 1: GND -> /GND
- C89 pad 1: /Bias-DAC/REF_P -> /REF_P
- C89 pad 2: /Bias-DAC/GND -> /GND
- C9 pad 1: +15V -> Net-(C9-Pad1)
- C9 pad 2: Net-(C10-Pad1) -> /GND
- C90 pad 1: /Bias-DAC/REF_N -> /REF_N
- C90 pad 2: /Bias-DAC/GND -> /GND
- C92 pad 1: /Bias-DAC/+15V -> /+15V
- C92 pad 2: /Bias-DAC/GND -> /GND
- C93 pad 1: /Bias-DAC/GND -> /GND
- C93 pad 2: /Bias-DAC/-15V -> /-15V
- C94 pad 1: /Bias-DAC/+15V -> /+15V
- C94 pad 2: /Bias-DAC/GND -> /GND
- C95 pad 1: /Bias-DAC/GND -> /GND
- C95 pad 2: /Bias-DAC/-15V -> /-15V
- C96 pad 1: /Bias-DAC/+15V -> /+15V
- C96 pad 2: /Bias-DAC/GND -> /GND
- C97 pad 1: /Bias-DAC/GND -> /GND
- C97 pad 2: /Bias-DAC/-15V -> /-15V
- C98 pad 1: /Bias-DAC/+15V -> /+15V
- C98 pad 2: /Bias-DAC/GND -> /GND
- C99 pad 1: /Bias-DAC/GND -> /GND
- C99 pad 2: /Bias-DAC/-15V -> /-15V
- J2 pad 1: -15V -> /-15V
- J2 pad 14: -15V -> /-15V
- J2 pad 15: GND -> /GND
- J2 pad 16: +15V -> /+15V
- J2 pad 18: GND -> /GND
- J2 pad 2: GND -> /GND
- J2 pad 21: GND -> /GND
- J2 pad 3: +15V -> /+15V
- J2 pad 5: GND -> /GND
- J2 pad 8: GND -> /GND
- R10 pad 2: GND -> /GND
- R19 pad 1: Net-(C13-Pad1) -> Net-(C9-Pad1)
- R20 pad 1: Net-(C14-Pad1) -> Net-(C10-Pad1)
- R9 pad 2: GND -> /GND
- U1 pad 2: GND -> /GND
- U10 pad 4: -15V -> /-15V
- U10 pad 7: +15V -> /+15V
- U11 pad 11: /Piezo-DACs/MISO -> /MISO
- U11 pad 12: /Piezo-DACs/MOSI -> /MOSI
- U11 pad 13: /Piezo-DACs/CLK -> /CLK
- U11 pad 15: GND -> /GND
- U11 pad 18: -15V -> /-15V
- U11 pad 19: GND -> /GND
- U11 pad 5: +15V -> /+15V
- U11 pad 8: /Piezo-DACs/~LDAC -> /~LDAC
- U12 pad 3: /Piezo-DACs/REF_P -> /REF_P
- U12 pad 4: -15V -> /-15V
- U12 pad 5: /Piezo-DACs/REF_N -> /REF_N
- U12 pad 8: +15V -> /+15V
- U13 pad 4: -15V -> /-15V
- U13 pad 7: +15V -> /+15V
- U15 pad P8_1: GND -> /GND
- U15 pad P8_2: GND -> /GND
- U15 pad P9_1: GND -> /GND
- U15 pad P9_2: GND -> /GND
- U15 pad P9_43: GND -> /GND
- U15 pad P9_44: GND -> /GND
- U15 pad P9_45: GND -> /GND
- U15 pad P9_46: GND -> /GND
- U16 pad 10: /Bias-DAC/3V3 -> /3V3
- U16 pad 11: /Bias-DAC/SDO -> /MISO
- U16 pad 12: /Bias-DAC/SDIN -> /MOSI
- U16 pad 13: /Bias-DAC/SCLK -> /CLK
- U16 pad 15: /Bias-DAC/GND -> /GND
- U16 pad 18: /Bias-DAC/-15V -> /-15V
- U16 pad 19: /Bias-DAC/GND -> /GND
- U16 pad 5: /Bias-DAC/+15V -> /+15V
- U16 pad 6: /Bias-DAC/3V3 -> /3V3
- U16 pad 7: /Bias-DAC/3V3 -> /3V3
- U16 pad 8: /Bias-DAC/~LDAC -> /~LDAC
- U16 pad 9: /Bias-DAC/3V3 -> /3V3
- U17 pad 3: /Bias-DAC/REF_P -> /REF_P
- U17 pad 4: /Bias-DAC/-15V -> /-15V
- U17 pad 5: /Bias-DAC/REF_N -> /REF_N
- U17 pad 8: /Bias-DAC/+15V -> /+15V
- U18 pad 4: /Bias-DAC/-15V -> /-15V
- U18 pad 7: /Bias-DAC/+15V -> /+15V
- U2 pad 2: GND -> /GND
- U3 pad 3: Net-(C13-Pad1) -> Net-(C9-Pad1)
- U3 pad 4: -15V -> /-15V
- U3 pad 5: Net-(C14-Pad1) -> Net-(C10-Pad1)
- U3 pad 8: +15V -> /+15V
- U4 pad 1: Net-(C20-Pad2) -> Net-(C20-Pad1)
- U4 pad 10: GND -> /GND
- U4 pad 15: +3V3 -> /3V3
- U4 pad 16: GND -> /GND
- U4 pad 3: GND -> /GND
- U4 pad 6: GND -> /GND
- U5 pad 11: /Piezo-DACs/MISO -> /MISO
- U5 pad 12: /Piezo-DACs/MOSI -> /MOSI
- U5 pad 13: /Piezo-DACs/CLK -> /CLK
- U5 pad 15: GND -> /GND
- U5 pad 18: -15V -> /-15V
- U5 pad 19: GND -> /GND
- U5 pad 5: +15V -> /+15V
- U5 pad 8: /Piezo-DACs/~LDAC -> /~LDAC
- U6 pad 3: /Piezo-DACs/REF_P -> /REF_P
- U6 pad 4: -15V -> /-15V
- U6 pad 5: /Piezo-DACs/REF_N -> /REF_N
- U6 pad 8: +15V -> /+15V
- U7 pad 4: -15V -> /-15V
- U7 pad 7: +15V -> /+15V
- U8 pad 11: /Piezo-DACs/MISO -> /MISO
- U8 pad 12: /Piezo-DACs/MOSI -> /MOSI
- U8 pad 13: /Piezo-DACs/CLK -> /CLK
- U8 pad 15: GND -> /GND
- U8 pad 18: -15V -> /-15V
- U8 pad 19: GND -> /GND
- U8 pad 5: +15V -> /+15V
- U8 pad 8: /Piezo-DACs/~LDAC -> /~LDAC
- U9 pad 3: /Piezo-DACs/REF_P -> /REF_P
- U9 pad 4: -15V -> /-15V
- U9 pad 5: /Piezo-DACs/REF_N -> /REF_N
- U9 pad 8: +15V -> /+15V
Routing:
- net /GND: track 0.00 -> 136.6 mm, vias 0 -> 129
- net /REF_P: track 0.00 -> 132.2 mm, vias 0 -> 6
- net /REF_N: track 0.00 -> 129.4 mm, vias 0 -> 6
- net /CLK: track 0.00 -> 121.1 mm, vias 0 -> 4
- net /MOSI: track 0.00 -> 115.8 mm, vias 0 -> 4
- net /MISO: track 0.00 -> 114.5 mm, vias 0 -> 4
- net /~LDAC: track 0.00 -> 101.1 mm, vias 0 -> 6
- net /+15V: track 0.00 -> 99.1 mm, vias 0 -> 42
- net /-15V: track 0.00 -> 92.9 mm, vias 0 -> 27
- net GND: track 76.5 -> 0.00 mm, vias 70 -> 0
- net /Piezo-DACs/REF_P: track 76.3 -> 0.00 mm, vias 3 -> 0
- net /Piezo-DACs/REF_N: track 75.9 -> 0.00 mm, vias 3 -> 0
- net /Piezo-DACs/CLK: track 71.1 -> 0.00 mm, vias 3 -> 0
- net /Piezo-DACs/~LDAC: track 68.9 -> 0.00 mm, vias 3 -> 0
- net /Piezo-DACs/MOSI: track 68.9 -> 0.00 mm, vias 3 -> 0
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- added copper zone on B.Cu, net /+15V
- added copper zone on F.Cu, net /+15V
- added copper zone on B.Cu, net /-15V
- added copper zone on F.Cu, net /-15V
- added copper zone on B.Cu, net /GND
- added copper zone on F.Cu, net /GND
- removed copper zone on B.Cu, net +15V
- removed copper zone on F.Cu, net +15V
- removed copper zone on B.Cu, net -15V
- removed copper zone on F.Cu, net -15V
- removed copper zone on B.Cu, net GND
- removed copper zone on F.Cu, net GND

Commit message: Reference schematic
Parts:
- removed J7: Conn_Coaxial, STM_Custom_Lib:SMA_horizontal
- added C106: 10u, Capacitor_SMD:C_0805_2012Metric_Pad1.15x1.40mm_HandSolder, F.Cu at (115.1, 75.2)
- added C107: 100n, Capacitor_SMD:C_0805_2012Metric_Pad1.15x1.40mm_HandSolder, F.Cu at (117.0, 75.2)
- added C108: 100n, Capacitor_SMD:C_0805_2012Metric_Pad1.15x1.40mm_HandSolder, F.Cu at (127.1, 76.5)
- added C109: 10u, Capacitor_SMD:C_0805_2012Metric_Pad1.15x1.40mm_HandSolder, F.Cu at (133.5, 76.5)
- added C110: opt, Capacitor_SMD:C_0805_2012Metric_Pad1.15x1.40mm_HandSolder, F.Cu at (140.5, 64.4)
- added C111: 100n, Capacitor_SMD:C_0805_2012Metric_Pad1.15x1.40mm_HandSolder, F.Cu at (145.6, 68.2)
- added C112: 100n, Capacitor_SMD:C_0805_2012Metric_Pad1.15x1.40mm_HandSolder, F.Cu at (136.7, 83.5)
- added C113: 10u, Capacitor_SMD:C_0805_2012Metric_Pad1.15x1.40mm_HandSolder, F.Cu at (147.5, 68.2)
- added C114: 10u, Capacitor_SMD:C_0805_2012Metric_Pad1.15x1.40mm_HandSolder, F.Cu at (136.7, 85.4)
- added C115: opt, Capacitor_SMD:C_0805_2012Metric_Pad1.15x1.40mm_HandSolder, F.Cu at (145.6, 79.7)
- added C116: 100n, Capacitor_SMD:C_0805_2012Metric_Pad1.15x1.40mm_HandSolder, F.Cu at (142.4, 75.9)
- added C117: 100n, Capacitor_SMD:C_0805_2012Metric_Pad1.15x1.40mm_HandSolder, F.Cu at (138.6, 74.0)
- added C118: 10u, Capacitor_SMD:C_0805_2012Metric_Pad1.15x1.40mm_HandSolder, F.Cu at (142.4, 74.0)
- added C119: 10u, Capacitor_SMD:C_0805_2012Metric_Pad1.15x1.40mm_HandSolder, F.Cu at (138.6, 75.9)
- added J5: Conn_Coaxial, Connector_Coaxial:SMB_Jack_Vertical, F.Cu at (129.7, 82.9)
- added R23: 1k5, Capacitor_SMD:C_0805_2012Metric_Pad1.15x1.40mm_HandSolder, F.Cu at (130.3, 75.2)
- added R24: 1k, Capacitor_SMD:C_0805_2012Metric_Pad1.15x1.40mm_HandSolder, F.Cu at (136.7, 66.3)
- added R25: 1k, Capacitor_SMD:C_0805_2012Metric_Pad1.15x1.40mm_HandSolder, F.Cu at (140.5, 83.5)
- added R26: 1k, Capacitor_SMD:C_0805_2012Metric_Pad1.15x1.40mm_HandSolder, F.Cu at (140.5, 66.3)
- added R27: 1k, Capacitor_SMD:C_0805_2012Metric_Pad1.15x1.40mm_HandSolder, F.Cu at (148.7, 81.0)
- added R28: 1k, Capacitor_SMD:C_0805_2012Metric_Pad1.15x1.40mm_HandSolder, F.Cu at (148.7, 78.4)
- added TP2: TestPoint, TestPoint:TestPoint_Loop_D1.80mm_Drill1.0mm_Beaded, F.Cu at (128.4, 72.1)
- added TP3: TestPoint, TestPoint:TestPoint_Loop_D1.80mm_Drill1.0mm_Beaded, F.Cu at (140.5, 86.7)
- added TP4: TestPoint, TestPoint:TestPoint_Loop_D1.80mm_Drill1.0mm_Beaded, F.Cu at (147.5, 72.1)
- added TP5: TestPoint, TestPoint:TestPoint_Loop_D1.80mm_Drill1.0mm_Beaded, F.Cu at (147.5, 75.2)
- added U19: ADP7142AUJZ-5.0, Package_TO_SOT_SMD:TSOT-23-5, F.Cu at (210.8, 116.0)
- added U20: ADR4550, Package_SO:SOIC-8_3.9x4.9mm_P1.27mm, F.Cu at (122.1, 74.6)
- added U21: AD8676, Package_SO:SOIC-8_3.9x4.9mm_P1.27mm, F.Cu at (140.5, 79.7)
- added U22: AD8675, Package_SO:SOIC-8_3.9x4.9mm_P1.27mm, F.Cu at (140.5, 70.2)
- C20: value 10u -> 2u2
- C21: value 100n -> 2u2; footprint Capacitor_SMD:C_0603_1608Metric_Pad1.05x0.95mm_HandSolder -> Capacitor_SMD:C_0805_2012Metric_Pad1.15x1.40mm_HandSolder
- J1: value Conn_Coaxial -> 609-5192-ND; footprint STM_Custom_Lib:SMA_horizontal -> STM_Custom_Lib:DSUB-9_Amphenol_LD09S33E4GV00LF
- R21, R22: value opt -> 0R
- moved N1 186.5 mm to (-109.7, -24.5), turned to 90 degrees
- moved A1 130.6 mm to (294.3, 72.7), turned to 270 degrees
- moved C18 87.4 mm to (199.8, 120.5), turned to 180 degrees
- moved R19 85.6 mm to (213.3, 104.2)
- moved R21 85.2 mm to (205.8, 115.2), turned to 90 degrees
- moved U4 80.8 mm to (204.8, 124.5), turned to 270 degrees
- moved R22 80.5 mm to (203.8, 115.2), turned to 90 degrees
- moved R20 74.3 mm to (213.3, 101.4)
- moved U3 69.1 mm to (204.8, 110.2), turned to 180 degrees
- moved C16 67.1 mm to (201.8, 115.2), turned to 90 degrees
- moved C17 66.3 mm to (204.8, 119.0), turned to 180 degrees
- moved C13 66.2 mm to (200.0, 111.2), turned to 90 degrees
- moved C11 65.9 mm to (198.2, 111.2), turned to 90 degrees
- moved C19 64.5 mm to (201.5, 124.0), turned to 270 degrees
- moved C9 63.0 mm to (213.3, 106.0)
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Connections:
- net /CLK renamed /DAC_CLK
- net /MISO renamed /DAC_MISO
- net /MOSI renamed /DAC_MOSI
- net /~CS-Bias renamed /~DAC_CS-Bias
- net /~CS-X renamed /~DAC_CS-X
- net /~CS-Y renamed /~DAC_CS-Y
- net /~CS-Z renamed /~DAC_CS-Z
- net /~LDAC renamed /~DAC_LDAC
- net Net-(A1-Pad2) renamed /Stepper-Driver/VDD
- net Net-(U4-Pad11) renamed /ADC_BUSY
- net Net-(U4-Pad12) renamed /ADC_MOSI
- net Net-(U4-Pad13) renamed /ADC_CLK
- net Net-(U4-Pad14) renamed /ADC_MISO
- net Net-(U4-Pad9) renamed /ADC_CONV
- A1 pad 1: Net-(A1-Pad1) -> /GND
- A1 pad 3: Net-(A1-Pad3) -> /Stepper-Driver/A+
- A1 pad 4: Net-(A1-Pad4) -> /Stepper-Driver/A-
- A1 pad 5: Net-(A1-Pad5) -> /Stepper-Driver/B+
- A1 pad 6: Net-(A1-Pad6) -> /Stepper-Driver/B-
- A1 pad 7: Net-(A1-Pad7) -> /GND
- A1 pad 8: Net-(A1-Pad8) -> /9V
- C21 pad 1: Net-(C20-Pad1) -> /GND
- C21 pad 2: /GND -> /+15V
- J1 pad 1: Net-(J1-Pad1) -> /+15V
- J1 pad 2: Net-(J1-Pad2) -> /GND
- J2 pad 10: Net-(J2-Pad10) -> /9V
- J2 pad 11: Net-(J2-Pad11) -> /GND
- J2 pad 23: Net-(J2-Pad10) -> /9V
- J2 pad 24: Net-(J2-Pad11) -> /GND
- J3 pad 0: GNDA -> /GND
- J3 pad 1: GNDA -> /GND
- J3 pad 2: GNDA -> /GND
- J3 pad 3: GNDA -> /GND
- J3 pad 4: GNDA -> /GND
- J3 pad 5: GNDA -> /GND
- J4 pad 0: GNDA -> /GND
- J4 pad 1: Net-(J4-Pad1) -> /GND
- J4 pad 2: Net-(J4-Pad2) -> /GND
- J4 pad 3: Net-(J4-Pad3) -> /GND
- J4 pad 4: Net-(J4-Pad4) -> /GND
- J4 pad 5: Net-(J4-Pad5) -> /GND
- J4 pad 6: Net-(J4-Pad6) -> /Stepper-Driver/B-
- J4 pad 7: Net-(J4-Pad7) -> /Stepper-Driver/B+
- J4 pad 8: Net-(J4-Pad8) -> /Stepper-Driver/A-
- J4 pad 9: Net-(J4-Pad9) -> /Stepper-Driver/A+
- JP1 pad 1: Net-(JP1-Pad1) -> Net-(C9-Pad1)
- JP1 pad 2: Net-(C15-Pad1) -> Net-(JP1-Pad2)
- JP2 pad 1: Net-(JP2-Pad1) -> Net-(C10-Pad1)
- JP2 pad 2: Net-(C16-Pad1) -> Net-(JP2-Pad2)
- R19 pad 2: /ADC/IN+ -> /ADC_IN+
- R20 pad 2: /ADC/IN- -> /ADC_IN-
- R21 pad 2: Net-(JP1-Pad1) -> Net-(R21-Pad2)
- R22 pad 2: Net-(JP2-Pad1) -> Net-(R22-Pad2)
- U3 pad 1: Net-(JP1-Pad1) -> Net-(R21-Pad2)
- U3 pad 2: Net-(JP1-Pad1) -> Net-(R21-Pad2)
- U3 pad 3: Net-(C9-Pad1) -> Net-(JP1-Pad2)
- U3 pad 5: Net-(C10-Pad1) -> Net-(JP2-Pad2)
- U3 pad 6: Net-(JP2-Pad1) -> Net-(R22-Pad2)
- U3 pad 7: Net-(JP2-Pad1) -> Net-(R22-Pad2)
Routing:
- net /DAC_MISO: track 114.5 -> 125.9 mm
- net /ADC/+5V: track 0.00 -> 10.1 mm
- net /+15V: track 99.1 -> 108.9 mm, vias 42 -> 50
- net Net-(JP2-Pad2): track 0.00 -> 9.49 mm
- net Net-(C16-Pad1): track 0.00 -> 8.45 mm
- net Net-(C15-Pad1): track 0.00 -> 8.45 mm
- net Net-(R22-Pad2): track 0.00 -> 7.94 mm
- net /ADC_IN-: track 0.00 -> 7.52 mm
- net /ADC_IN+: track 0.00 -> 7.52 mm
- net /GND: track 136.6 -> 143.9 mm, vias 129 -> 131
- net Net-(JP1-Pad2): track 0.00 -> 6.73 mm
- net /3V3: track 137.6 -> 143.8 mm, vias 0 -> 1
- net Net-(R21-Pad2): track 0.00 -> 6.08 mm
- net Net-(C9-Pad1): track 0.00 -> 5.49 mm
- net Net-(C10-Pad1): track 0.00 -> 5.19 mm
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
Commit message: Layout progress
Parts:
- removed J5: Conn_Coaxial, Connector_Coaxial:SMB_Jack_Vertical
- added TP6: TestPoint, TestPoint:TestPoint_Loop_D1.80mm_Drill1.0mm_Beaded, F.Cu at (132.9, 87.3)
- moved N1 288.0 mm to (150.0, 100.0)
- moved A1 144.7 mm to (174.1, 153.3), turned to 90 degrees
- moved C106 16.7 mm to (130.9, 70.2), turned to 180 degrees
- moved C107 14.3 mm to (130.9, 72.1), turned to 180 degrees
- moved TP2 13.1 mm to (129.3, 85.1)
- moved U20 9.86 mm to (131.6, 77.1), turned to 270 degrees
- moved R23 7.67 mm to (133.5, 82.2)
- moved C109 7.62 mm to (133.5, 84.1), turned to 180 degrees
- moved C108 6.25 mm to (129.7, 82.2), turned to 180 degrees
- moved TP4 6.02 mm to (149.4, 77.8)
- moved C110 5.72 mm to (140.5, 70.2)
- moved C111 5.72 mm to (145.6, 74.0)
- moved C112 5.72 mm to (136.7, 89.2)
- moved C113 5.72 mm to (147.5, 74.0)
- moved C114 5.72 mm to (136.7, 91.1)
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Routing:
- net /REF_P: track 132.2 -> 157.1 mm, vias 6 -> 5
- net /+15V: track 108.9 -> 127.0 mm, vias 50 -> 61
- net Net-(C109-Pad1): track 0.00 -> 17.4 mm
- net Net-(R25-Pad2): track 0.00 -> 14.0 mm
- net /3V3: track 143.8 -> 156.8 mm, vias 1 -> 5
- net /REF_N: track 129.4 -> 141.3 mm, vias 6 -> 5
- net /-15V: track 97.0 -> 107.3 mm, vias 33 -> 42
- net Net-(C115-Pad1): track 0.00 -> 9.82 mm
- net Net-(C110-Pad1): track 0.00 -> 8.47 mm
- net /DAC_MISO: track 125.9 -> 134.3 mm
- net Net-(C108-Pad1): track 0.00 -> 7.97 mm
- net /GND: track 143.9 -> 148.9 mm, vias 131 -> 160
- net /DAC_MOSI: track 115.8 -> 120.0 mm
- net /DAC_CLK: track 121.1 -> 125.3 mm
- net /~DAC_LDAC: track 101.1 -> 105.3 mm
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- added copper zone on F.Cu, net /+20V
- added copper zone on F.Cu, net /-20V
- added copper zone on B.Cu, net /3V3
Other:
- board size 160 x 120 mm -> 164.2 x 120 mm

Commit message: Reference layout finished
Parts:
- moved N1 266.5 mm to (-70.3, -49.9)
- moved TP1 117.6 mm to (214.0, 119.5)
- moved C80 114.0 mm to (208.2, 48.0)
- moved C79 112.0 mm to (197.1, 48.0)
- moved C78 25.0 mm to (116.2, 66.2)
- moved C77 21.6 mm to (103.5, 65.5)
- moved TP5 19.0 mm to (139.2, 63.8)
- moved TP4 15.3 mm to (144.9, 63.2)
- moved A1 10.9 mm to (185.0, 154.5)
- moved U15 1.90 mm to (71.9, 155.9)
- moved C25 0.75 mm to (209.2, 130.2)
Connections:
- net Net-(A1-Pad15) renamed /Stepper-Driver/STEP
- net Net-(A1-Pad16) renamed /Stepper-Driver/DIR
- net Net-(A1-Pad9) renamed /Stepper-Driver/~ENABLE
- A1 pad 2: /Stepper-Driver/VDD -> /3V3
- TP1 pad 1: Net-(TP1-Pad1) -> /ADC/+5V
Routing:
- net /~DAC_CS-X: track 21.7 -> 95.5 mm, vias 0 -> 1
- net /~DAC_CS-Z: track 39.6 -> 99.0 mm, vias 0 -> 1
- net /ADC_MISO: track 3.06 -> 55.2 mm
- net /3V3: track 156.8 -> 208.3 mm, vias 5 -> 6
- net /ADC_CLK: track 2.85 -> 53.8 mm
- net /ADC_MOSI: track 3.06 -> 52.5 mm
- net /ADC_BUSY: track 3.26 -> 51.3 mm
- net /ADC_CONV: track 3.26 -> 49.8 mm
- net (no net): track 0.00 -> 44.3 mm
- net /~DAC_CS-Y: track 39.6 -> 73.7 mm, vias 0 -> 1
- net /~DAC_CS-Bias: track 17.8 -> 36.0 mm, vias 0 -> 1
- net /REF_N: track 141.3 -> 155.1 mm
- net /DAC_CLK: track 125.3 -> 115.0 mm
- net /REF_P: track 157.1 -> 166.7 mm
- net /DAC_MOSI: track 120.0 -> 111.0 mm
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Other:
- board size 164.2 x 120 mm -> 160 x 120 mm
