File: Electronics/Mainboard/Mainboard.kicad_pcb (KiCad board)
At the start: 2 copper layers, 160 x 120 mm, 193 parts, among them J1 609-5192-ND, J2 DB25_Male_MountingHoles, J3 609-5192-ND, J4 609-5192-ND, U1 AD8676, U10 AD8675, U11 AD5781, U12 AD8676xR, U13 AD8675, U14 LM75C, U15 Beaglebone_Black, U16 AD5781, U17 AD8676xR, U18 AD8675, U19 ADP7142AUJZ-5.0, U2 AD8676, U20 ADR4550, U21 AD8676, U22 AD8675, U3 LT1469, U4 LTC2338-18, U5 AD5781, U6 AD8676xR, U7 AD8675, U8 AD5781, U9 AD8676xR

Commit message: Layout nearly finished
Parts:
- added C122: 1u, Capacitor_SMD:C_1210_3225Metric_Pad1.42x2.65mm_HandSolder, B.Cu at (164.6, 55.8)
- added C123: 1u, Capacitor_SMD:C_1210_3225Metric_Pad1.42x2.65mm_HandSolder, B.Cu at (155.5, 62.6)
- added C124: 1u, Capacitor_SMD:C_1210_3225Metric_Pad1.42x2.65mm_HandSolder, B.Cu at (164.3, 128.3)
- added C125: 1u, Capacitor_SMD:C_1210_3225Metric_Pad1.42x2.65mm_HandSolder, B.Cu at (184.4, 111.7)
- added C126: 1u, Capacitor_SMD:C_1210_3225Metric_Pad1.42x2.65mm_HandSolder, B.Cu at (179.6, 76.6)
- added C127: 1u, Capacitor_SMD:C_1210_3225Metric_Pad1.42x2.65mm_HandSolder, B.Cu at (187.7, 123.1)
- added C128: 1u, Capacitor_SMD:C_1210_3225Metric_Pad1.42x2.65mm_HandSolder, B.Cu at (135.1, 84.1)
- added C129: 1u, Capacitor_SMD:C_1210_3225Metric_Pad1.42x2.65mm_HandSolder, B.Cu at (173.7, 50.0)
- added C130: 1u, Capacitor_SMD:C_1210_3225Metric_Pad1.42x2.65mm_HandSolder, B.Cu at (194.2, 82.8)
- added C131: 1u, Capacitor_SMD:C_1210_3225Metric_Pad1.42x2.65mm_HandSolder, B.Cu at (187.7, 73.3)
- added C132: 1u, Capacitor_SMD:C_1210_3225Metric_Pad1.42x2.65mm_HandSolder, B.Cu at (179.2, 129.9)
- added C133: 1u, Capacitor_SMD:C_1210_3225Metric_Pad1.42x2.65mm_HandSolder, B.Cu at (194.2, 124.0)
- added C134: 1u, Capacitor_SMD:C_1210_3225Metric_Pad1.42x2.65mm_HandSolder, B.Cu at (215.3, 102.3)
- added C135: 1u, Capacitor_SMD:C_1210_3225Metric_Pad1.42x2.65mm_HandSolder, B.Cu at (139.3, 73.7)
- added C136: 1u, Capacitor_SMD:C_1210_3225Metric_Pad1.42x2.65mm_HandSolder, B.Cu at (202.7, 119.8)
- added C137: 1u, Capacitor_SMD:C_1210_3225Metric_Pad1.42x2.65mm_HandSolder, B.Cu at (209.8, 96.1)
- added C138: 100n, Capacitor_SMD:C_0603_1608Metric_Pad1.05x0.95mm_HandSolder, F.Cu at (114.4, 93.0)
- added JP11: Jumper_NC_Dual, Jumper:SolderJumper-3_P2.0mm_Open_TrianglePad1.0x1.5mm, F.Cu at (101.1, 97.5)
- added R29: 4k7, Capacitor_SMD:C_0805_2012Metric_Pad1.15x1.40mm_HandSolder, F.Cu at (117.6, 87.9)
- added TP10: TestPoint, TestPoint:TestPoint_Loop_D1.80mm_Drill1.0mm_Beaded, F.Cu at (97.0, 44.1)
- added TP11: TestPoint, TestPoint:TestPoint_Loop_D1.80mm_Drill1.0mm_Beaded, F.Cu at (120.2, 97.5)
- added TP12: TestPoint, TestPoint:TestPoint_Loop_D1.80mm_Drill1.0mm_Beaded, F.Cu at (178.6, 141.9)
- added TP13: TestPoint, TestPoint:TestPoint_Loop_D1.80mm_Drill1.0mm_Beaded, F.Cu at (86.5, 76.5)
- added TP7: TestPoint, TestPoint:TestPoint_Loop_D1.80mm_Drill1.0mm_Beaded, F.Cu at (97.0, 51.9)
- added TP8: TestPoint, TestPoint:TestPoint_Loop_D1.80mm_Drill1.0mm_Beaded, F.Cu at (97.0, 59.7)
- added TP9: TestPoint, TestPoint:TestPoint_Loop_D1.80mm_Drill1.0mm_Beaded, F.Cu at (104.2, 48.0)
- TP4, TP5: footprint TestPoint:TestPoint_Loop_D1.80mm_Drill1.0mm_Beaded -> TestPoint:TestPoint_Pad_D2.0mm
- moved U14 70.4 mm to (113.8, 87.9), turned to 270 degrees
- moved TP4 27.8 mm to (144.3, 70.2)
- moved N1 25.5 mm to (-60.3, -26.4)
- moved TP5 23.7 mm to (158.9, 82.2)
- moved C81 21.7 mm to (96.0, 73.3)
- moved C121 0.64 mm to (96.0, 92.4)
- moved C82 0.63 mm to (96.0, 82.9)
- moved C120 0.38 mm to (183.7, 142.5)
Connections:
- net Net-(J2-Pad0) renamed /Shield
- C81 pad 1: /3V3 -> /Power/digital_3V3
- J2 pad 12: Net-(J2-Pad12) -> /i2c_scl
- J2 pad 13: Net-(J2-Pad13) -> /i2c_sda
- J2 pad 20: /3V3 -> /Power/digital_3V3
- J2 pad 7: /3V3 -> /Power/digital_3V3
- U14 pad 1: Net-(U14-Pad1) -> /i2c_sda
- U14 pad 2: Net-(U14-Pad2) -> /i2c_scl
- U14 pad 4: Net-(U14-Pad4) -> /GND
- U14 pad 5: Net-(U14-Pad5) -> /GND
- U14 pad 6: Net-(U14-Pad5) -> /GND
- U14 pad 7: Net-(U14-Pad7) -> /3V3
- U14 pad 8: Net-(U14-Pad8) -> /3V3
- U15 pad P9_19: Net-(U15-PadP9_19) -> /i2c_scl
- U15 pad P9_20: Net-(U15-PadP9_20) -> /i2c_sda
- U15 pad P9_3: Net-(U15-PadP9_3) -> /Beaglebone/3V3
Routing:
- net /i2c_sda: track 0.00 -> 63.3 mm, vias 0 -> 1
- net /i2c_scl: track 0.00 -> 57.9 mm, vias 0 -> 1
- net /Power/digital_3V3: track 0.00 -> 24.7 mm, vias 0 -> 4
- net /GND: track 186.6 -> 199.6 mm, vias 216 -> 251
- net /Beaglebone/3V3: track 0.00 -> 9.64 mm
- net /3V3: track 215.7 -> 224.9 mm, vias 6 -> 9
- net /5V: track 3.16 -> 7.44 mm, vias 0 -> 6
- net /REF_P: track 155.3 -> 158.1 mm
- net /REF_N: track 146.7 -> 148.6 mm
- net /Bias-DAC/GND: vias 1 -> 0
- net /9V: vias 0 -> 5
- added copper zone on F.Cu, net /3V3
- added copper zone on F.Cu, net /5V
- added copper zone on B.Cu, net /9V
- added copper zone on B.Cu, net /Power/digital_3V3
- added copper zone on F.Cu, net /Power/digital_3V3
- added copper zone on B.Cu, net /Shield
- added copper zone on F.Cu, net /Shield

Commit message: Silkscreen rearanged
Parts:
- added C139: C_Small, Capacitor_SMD:C_1206_3216Metric_Pad1.42x1.75mm_HandSolder, F.Cu at (220.8, 44.1)
- added JP12: Jumper, Jumper:SolderJumper-2_P1.3mm_Open_TrianglePad1.0x1.5mm, F.Cu at (225.8, 46.0)
- added R30: R_Small, Resistor_SMD:R_1206_3216Metric_Pad1.42x1.75mm_HandSolder, F.Cu at (220.8, 46.7)
Routing:
- net Net-(C139-Pad2): track 0.00 -> 6.34 mm
- net /GND: track 199.6 -> 202.5 mm, vias 251 -> 253
- net /Shield: track 0.00 -> 2.17 mm, vias 0 -> 10
Other:
- board text added: "+15V"
- board text added: "+20V"
- board text added: "+3.3V"
- board text added: "+REF"
- board text added: "-15V"
- board text added: "-20V"
- board text added: "-REF"

Commit message: Mainboard layout and schematic done
Parts:
- added C140: 1n, Capacitor_SMD:C_0603_1608Metric_Pad1.05x0.95mm_HandSolder, F.Cu at (206.5, 105.5)
- added C141: 680p, Capacitor_SMD:C_0603_1608Metric_Pad1.05x0.95mm_HandSolder, F.Cu at (202.0, 106.5)
- added JP13: Jumper, Jumper:SolderJumper-2_P1.3mm_Bridged_RoundedPad1.0x1.5mm, B.Cu at (129.7, 112.1)
- added JP14: Jumper, Jumper:SolderJumper-2_P1.3mm_Bridged_RoundedPad1.0x1.5mm, B.Cu at (132.2, 112.1)
- added JP15: Jumper, Jumper:SolderJumper-2_P1.3mm_Bridged_RoundedPad1.0x1.5mm, B.Cu at (127.1, 112.1)
- added JP16: Jumper, Jumper:SolderJumper-2_P1.3mm_Bridged_RoundedPad1.0x1.5mm, B.Cu at (124.6, 148.3)
- added JP17: Jumper, Jumper:SolderJumper-2_P1.3mm_Bridged_RoundedPad1.0x1.5mm, B.Cu at (127.1, 148.3)
- added JP18: Jumper, Jumper:SolderJumper-2_P1.3mm_Bridged_RoundedPad1.0x1.5mm, B.Cu at (139.8, 148.3)
- added JP19: Jumper, Jumper:SolderJumper-2_P1.3mm_Bridged_RoundedPad1.0x1.5mm, B.Cu at (142.4, 148.3)
- added JP20: Jumper, Jumper:SolderJumper-2_P1.3mm_Bridged_RoundedPad1.0x1.5mm, B.Cu at (144.9, 148.3)
- added JP21: Jumper, Jumper:SolderJumper-2_P1.3mm_Bridged_RoundedPad1.0x1.5mm, B.Cu at (147.5, 148.3)
- added JP22: Jumper, Jumper:SolderJumper-2_P1.3mm_Bridged_RoundedPad1.0x1.5mm, B.Cu at (125.9, 156.5)
- added JP23: Jumper, Jumper:SolderJumper-2_P1.3mm_Bridged_RoundedPad1.0x1.5mm, B.Cu at (141.1, 156.5)
- added JP24: Jumper, Jumper:SolderJumper-2_P1.3mm_Bridged_RoundedPad1.0x1.5mm, B.Cu at (150.6, 155.9)
- added JP25: Jumper, Jumper:SolderJumper-2_P1.3mm_Bridged_RoundedPad1.0x1.5mm, B.Cu at (150.6, 152.1)
- added JP26: Jumper, Jumper:SolderJumper-2_P1.3mm_Bridged_RoundedPad1.0x1.5mm, B.Cu at (154.4, 154.0)
- added JP27: Jumper, Jumper:SolderJumper-2_P1.3mm_Bridged_RoundedPad1.0x1.5mm, B.Cu at (115.1, 98.1)
- added JP28: Jumper, Jumper:SolderJumper-2_P1.3mm_Bridged_RoundedPad1.0x1.5mm, B.Cu at (112.5, 98.1)
- added JP29: Jumper, Jumper:SolderJumper-2_P1.3mm_Open_TrianglePad1.0x1.5mm, B.Cu at (226.1, 44.7)
- added LOGO1: Logo_Open_Hardware_Small, Symbol:OSHW-Logo2_24.3x20mm_SilkScreen, B.Cu at (111.6, 61.2)
- added R31: 1k, Resistor_SMD:R_0603_1608Metric_Pad1.05x0.95mm_HandSolder, F.Cu at (211.2, 109.8)
- added R32: 1k, Resistor_SMD:R_0603_1608Metric_Pad1.05x0.95mm_HandSolder, F.Cu at (204.8, 105.5)
- added SYM1: SYM_ESD_Large, Symbol:ESD-Logo_13.2x12mm_SilkScreen, B.Cu at (203.8, 132.0)
- added TP14: TestPoint, TestPoint:TestPoint_Pad_D1.5mm, F.Cu at (215.5, 112.8)
- added TP15: TestPoint, TestPoint:TestPoint_Pad_D1.5mm, F.Cu at (208.8, 90.0)
- added TP16: TestPoint, TestPoint:TestPoint_Pad_D1.5mm, F.Cu at (206.5, 92.0)
- added TP17: TestPoint, TestPoint:TestPoint_Pad_D1.5mm, B.Cu at (100.5, 100.6)
- added TP18: TestPoint, TestPoint:TestPoint_Pad_D1.5mm, B.Cu at (103.0, 100.6)
- added TP19: TestPoint, TestPoint:TestPoint_Pad_D1.5mm, B.Cu at (105.5, 100.6)
- added TP20: TestPoint, TestPoint:TestPoint_Pad_D1.5mm, B.Cu at (108.1, 100.6)
- added TP21: TestPoint, TestPoint:TestPoint_Pad_D1.5mm, B.Cu at (110.6, 100.6)
- added TP22: TestPoint, TestPoint:TestPoint_Pad_D1.5mm, B.Cu at (118.2, 100.6)
- added TP23: TestPoint, TestPoint:TestPoint_Pad_D1.5mm, B.Cu at (120.8, 100.6)
- added TP24: TestPoint, TestPoint:TestPoint_Pad_D1.5mm, B.Cu at (132.2, 100.6)
- added TP25: TestPoint, TestPoint:TestPoint_Pad_D1.5mm, B.Cu at (134.8, 100.6)
- added TP26: TestPoint, TestPoint:TestPoint_Pad_D1.5mm, B.Cu at (137.3, 100.6)
- added TP27: TestPoint, TestPoint:TestPoint_Pad_D1.5mm, B.Cu at (139.8, 100.6)
- added TP28: TestPoint, TestPoint:TestPoint_Pad_D1.5mm, B.Cu at (142.4, 100.6)
- added TP29: TestPoint, TestPoint:TestPoint_Pad_D1.5mm, B.Cu at (101.7, 108.9)
- added TP30: TestPoint, TestPoint:TestPoint_Pad_D1.5mm, B.Cu at (104.3, 108.9)
- added TP31: TestPoint, TestPoint:TestPoint_Pad_D1.5mm, B.Cu at (106.8, 108.9)
- added TP32: TestPoint, TestPoint:TestPoint_Pad_D1.5mm, B.Cu at (109.4, 108.9)
- added TP33: TestPoint, TestPoint:TestPoint_Pad_D1.5mm, B.Cu at (111.9, 108.9)
- added TP34: TestPoint, TestPoint:TestPoint_Pad_D1.5mm, B.Cu at (115.1, 108.9)
- added TP35: TestPoint, TestPoint:TestPoint_Pad_D1.5mm, B.Cu at (117.6, 108.9)
- added TP36: TestPoint, TestPoint:TestPoint_Pad_D1.5mm, B.Cu at (120.2, 108.9)
- added TP37: TestPoint, TestPoint:TestPoint_Pad_D1.5mm, B.Cu at (124.0, 109.1)
- added TP38: TestPoint, TestPoint:TestPoint_Pad_D1.5mm, B.Cu at (130.3, 109.1)
- added TP39: TestPoint, TestPoint:TestPoint_Pad_D1.5mm, B.Cu at (134.1, 108.9)
- added TP40: TestPoint, TestPoint:TestPoint_Pad_D1.5mm, B.Cu at (136.7, 108.9)
- added TP41: TestPoint, TestPoint:TestPoint_Pad_D1.5mm, B.Cu at (139.2, 108.9)
- added TP42: TestPoint, TestPoint:TestPoint_Pad_D1.5mm, B.Cu at (141.7, 108.9)
- added TP43: TestPoint, TestPoint:TestPoint_Pad_D1.5mm, B.Cu at (144.3, 108.9)
- added TP44: TestPoint, TestPoint:TestPoint_Pad_D1.5mm, B.Cu at (94.1, 148.9)
- added TP45: TestPoint, TestPoint:TestPoint_Pad_D1.5mm, B.Cu at (96.7, 148.9)
- added TP46: TestPoint, TestPoint:TestPoint_Pad_D1.5mm, B.Cu at (99.2, 148.9)
- added TP47: TestPoint, TestPoint:TestPoint_Pad_D1.5mm, B.Cu at (101.7, 148.9)
- added TP48: TestPoint, TestPoint:TestPoint_Pad_D1.5mm, B.Cu at (104.3, 148.9)
- added TP49: TestPoint, TestPoint:TestPoint_Pad_D1.5mm, B.Cu at (106.8, 148.9)
- added TP50: TestPoint, TestPoint:TestPoint_Pad_D1.5mm, B.Cu at (109.4, 148.9)
- added TP51: TestPoint, TestPoint:TestPoint_Pad_D1.5mm, B.Cu at (111.9, 148.9)
- added TP52: TestPoint, TestPoint:TestPoint_Pad_D1.5mm, B.Cu at (114.4, 148.9)
- added TP53: TestPoint, TestPoint:TestPoint_Pad_D1.5mm, B.Cu at (117.0, 148.9)
- added TP54: TestPoint, TestPoint:TestPoint_Pad_D1.5mm, B.Cu at (119.5, 148.9)
- added TP55: TestPoint, TestPoint:TestPoint_Pad_D1.5mm, B.Cu at (122.1, 148.9)
- added TP56: TestPoint, TestPoint:TestPoint_Pad_D1.5mm, B.Cu at (99.2, 108.9)
- added TP57: TestPoint, TestPoint:TestPoint_Pad_D1.5mm, B.Cu at (132.2, 148.9)
- added TP58: TestPoint, TestPoint:TestPoint_Pad_D1.5mm, B.Cu at (134.8, 148.9)
- added TP59: TestPoint, TestPoint:TestPoint_Pad_D1.5mm, B.Cu at (137.3, 148.9)
- added TP60: TestPoint, TestPoint:TestPoint_Pad_D1.5mm, B.Cu at (92.8, 155.9)
- added TP61: TestPoint, TestPoint:TestPoint_Pad_D1.5mm, B.Cu at (95.4, 155.9)
- added TP62: TestPoint, TestPoint:TestPoint_Pad_D1.5mm, B.Cu at (97.9, 155.9)
- added TP63: TestPoint, TestPoint:TestPoint_Pad_D1.5mm, B.Cu at (100.5, 155.9)
- added TP64: TestPoint, TestPoint:TestPoint_Pad_D1.5mm, B.Cu at (103.0, 155.9)
- added TP65: TestPoint, TestPoint:TestPoint_Pad_D1.5mm, B.Cu at (105.5, 155.9)
- added TP66: TestPoint, TestPoint:TestPoint_Pad_D1.5mm, B.Cu at (108.1, 155.9)
- added TP67: TestPoint, TestPoint:TestPoint_Pad_D1.5mm, B.Cu at (110.6, 155.9)
- added TP68: TestPoint, TestPoint:TestPoint_Pad_D1.5mm, B.Cu at (113.2, 155.9)
- added TP69: TestPoint, TestPoint:TestPoint_Pad_D1.5mm, B.Cu at (115.7, 155.9)
- added TP70: TestPoint, TestPoint:TestPoint_Pad_D1.5mm, B.Cu at (118.2, 155.9)
- added TP71: TestPoint, TestPoint:TestPoint_Pad_D1.5mm, B.Cu at (120.8, 155.9)
- added TP73: TestPoint, TestPoint:TestPoint_Pad_D1.5mm, B.Cu at (130.3, 156.5)
- added TP74: TestPoint, TestPoint:TestPoint_Pad_D1.5mm, B.Cu at (132.9, 156.5)
- added TP75: TestPoint, TestPoint:TestPoint_Pad_D1.5mm, B.Cu at (135.4, 156.5)
- added TP76: TestPoint, TestPoint:TestPoint_Pad_D1.5mm, B.Cu at (137.9, 156.5)
- C10: value 66n -> 680p
- C107, C108, C111, C112, C116, C117: footprint Capacitor_SMD:C_0805_2012Metric_Pad1.15x1.40mm_HandSolder -> Capacitor_SMD:C_0603_1608Metric_Pad1.05x0.95mm_HandSolder
- C122, C123, C124, C125, C126, C127, C128, C129, C130, C131, C132, C133, C134, C135, C136, C137: value 1u -> 10u; footprint Capacitor_SMD:C_1210_3225Metric_Pad1.42x2.65mm_HandSolder -> Capacitor_SMD:C_1206_3216Metric
- C139: value C_Small -> 100n
- C83, C84, C85, C86, C87, C88: value opt -> 220p
- C9: value 66n -> 1n
- JP1, JP2: footprint Connector_PinHeader_2.54mm:PinHeader_1x02_P2.54mm_Vertical -> Jumper:SolderJumper-2_P1.3mm_Bridged_RoundedPad1.0x1.5mm; moved to B.Cu
- R1, R10, R11, R12, R13, R14, R2, R24, R25, R26, R27, R28, R29, R3, R4, R5, R6, R7, R8, R9: footprint Capacitor_SMD:C_0805_2012Metric_Pad1.15x1.40mm_HandSolder -> Resistor_SMD:R_0805_2012Metric
- R15, R16, R17, R18: value 220 -> 49R9; footprint Capacitor_SMD:C_0805_2012Metric_Pad1.15x1.40mm_HandSolder -> Resistor_SMD:R_0805_2012Metric
- R19, R20: value 50R -> 560R; footprint Resistor_SMD:R_0805_2012Metric_Pad1.15x1.40mm_HandSolder -> Resistor_SMD:R_0603_1608Metric_Pad1.05x0.95mm_HandSolder
- R21, R22: footprint Resistor_SMD:R_0805_2012Metric_Pad1.15x1.40mm_HandSolder -> Resistor_SMD:R_0805_2012Metric
- R23: value 1k5 -> 1k; footprint Capacitor_SMD:C_0805_2012Metric_Pad1.15x1.40mm_HandSolder -> Resistor_SMD:R_0805_2012Metric
- R30: value R_Small -> 1M2
- moved JP1 88.0 mm to (122.1, 112.1), turned to 90 degrees
- moved JP2 85.8 mm to (124.6, 112.1), turned to 90 degrees
- moved C137 16.3 mm to (213.2, 112.0)
- moved C10 9.11 mm to (211.2, 108.2)
- moved C9 5.99 mm to (211.2, 111.2)
- moved C134 5.42 mm to (210.0, 101.2), turned to 180 degrees
- moved C12 4.19 mm to (210.8, 105.2), turned to 270 degrees
- moved C14 4.04 mm to (208.8, 105.5), turned to 270 degrees
- moved R19 0.70 mm to (214.8, 104.2)
- moved R20 0.70 mm to (214.8, 101.4)
Connections:
- C9 pad 2: /GND -> Net-(C9-Pad2)
- JP1 pad 1: Net-(C9-Pad1) -> /ADC_MISO
- JP2 pad 1: Net-(C10-Pad1) -> /ADC_CLK
- R19 pad 1: Net-(C9-Pad1) -> Net-(C9-Pad2)
- R20 pad 1: Net-(C10-Pad1) -> Net-(C140-Pad2)
- R21 pad 2: Net-(R21-Pad2) -> Net-(C9-Pad1)
- U15 pad P8_27: /Stepper-Driver/DIR -> Net-(JP16-Pad2)
- U15 pad P8_28: /Stepper-Driver/~ENABLE -> Net-(JP22-Pad1)
- U15 pad P8_29: /Beaglebone/Motor-Step -> Net-(JP17-Pad2)
- U15 pad P8_39: /~DAC_CS-Bias -> Net-(JP18-Pad2)
- U15 pad P8_40: /~DAC_LDAC -> Net-(JP23-Pad1)
- U15 pad P8_41: /~DAC_CS-Y -> Net-(JP19-Pad2)
- U15 pad P8_42: /DAC_CLK -> Net-(JP24-Pad1)
- U15 pad P8_43: /~DAC_CS-Z -> Net-(JP20-Pad2)
- U15 pad P8_44: /DAC_MISO -> Net-(JP25-Pad1)
- U15 pad P8_45: /~DAC_CS-X -> Net-(JP21-Pad2)
- U15 pad P8_46: /DAC_MOSI -> Net-(JP26-Pad1)
- U15 pad P9_19: /i2c_scl -> Net-(JP27-Pad2)
- U15 pad P9_20: /i2c_sda -> Net-(JP28-Pad1)
- U15 pad P9_25: /ADC_MISO -> Net-(JP1-Pad2)
- U15 pad P9_27: /ADC_CLK -> Net-(JP2-Pad2)
- U15 pad P9_29: /ADC_BUSY -> Net-(JP13-Pad2)
- U15 pad P9_30: /ADC_MOSI -> Net-(JP15-Pad1)
- U15 pad P9_31: /ADC_CONV -> Net-(JP14-Pad2)
- U3 pad 1: Net-(R21-Pad2) -> Net-(C9-Pad1)
- U3 pad 2: Net-(R21-Pad2) -> Net-(C9-Pad1)
- U3 pad 3: Net-(JP1-Pad2) -> Net-(C10-Pad1)
- U3 pad 5: Net-(JP2-Pad2) -> Net-(C141-Pad1)
Routing:
- net Net-(C140-Pad2): track 0.00 -> 11.0 mm
- net /DAC_CLK: track 159.1 -> 148.6 mm
- net /ADC_MISO: track 126.4 -> 116.9 mm
- net /ADC_CLK: track 122.1 -> 112.6 mm
- net /ADC_BUSY: track 115.0 -> 105.4 mm
- net /ADC_CONV: track 111.7 -> 102.2 mm
- net Net-(C9-Pad2): track 0.00 -> 9.50 mm
- net Net-(JP13-Pad2): track 0.00 -> 9.29 mm
- net Net-(JP14-Pad2): track 0.00 -> 9.29 mm
- net Net-(JP24-Pad1): track 0.00 -> 8.39 mm
- net /i2c_sda: track 63.3 -> 55.0 mm
- net Net-(JP28-Pad1): track 0.00 -> 7.76 mm
- net /DAC_MOSI: track 146.1 -> 138.5 mm
- net /ADC_MOSI: track 115.5 -> 108.5 mm
- net /DAC_MISO: track 168.9 -> 162.3 mm
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Other:
- outline, holes or cut-outs redrawn
- board text added: "BOT"
- board text added: "STM Mainboard V1"
- board text added: "TOP"
- board text added: "©mr.kenhoff 2020"

Commit message: Head interconnect finished
Parts:
- moved N1 245.2 mm to (149.8, 100.0)
Routing:
- net /Shield: vias 10 -> 18
- net /GND: vias 261 -> 275
- net /-15V: vias 62 -> 65
Other:
- board text added: "ADC SPI"
- board text added: "BUSY"
- board text added: "Beaglebone 3.3V"
- board text added: "CLK"
- board text added: "CONV"
- board text added: "CS Bias"
- board text added: "CS X"
- board text added: "CS Y"
- board text added: "CS Z"
- board text added: "DAC CLK"
- board text added: "DAC MISO"
- board text added: "DAC MOSI"
- board text added: "Dir"
- board text added: "EN"
- board text added: "Ext. 3.3V"
- board text added: "LDAC"
- board text added: "MISO"
- board text added: "MOSI"
- board text added: "SCL"
- board text added: "SDA"
- board text added: "Step"
- board text added: "Stepper Driver"
- board text added: "©mrkenhoff 2020"
- board text removed: "©mr.kenhoff 2020"

Commit message: Added images
Parts:
- C120: value 100u 35V -> 220u 16V
- C121, C81, C82: value 330u 16V -> 330u 25V
- C77, C78, C79, C80: value 220u 25V -> 330u 25V
- U1, U2: value AD8676 -> OPA2991
- U12, U17, U6, U9: value AD8676xR -> AD8676
