File: Electronics/Mainboard/ADC.sch (KiCad schematic (older format))
At the start: 0 parts

Commit message: Supply board and tunneling amp finished
Parts:
- added C10, C19, C21, C22, C24, C9: 100n, Capacitor_SMD:C_0805_2012Metric_Pad1.15x1.40mm_HandSolder, symbol Device:C
- added C11, C12, C20, C23, C25: 10u, Capacitor_SMD:C_1206_3216Metric_Pad1.42x1.75mm_HandSolder, symbol Device:C
- added C13, C14: 66n, Capacitor_SMD:C_0805_2012Metric_Pad1.15x1.40mm_HandSolder, symbol Device:C
- added C15, C16, C17: opt, Capacitor_SMD:C_0805_2012Metric_Pad1.15x1.40mm_HandSolder, symbol Device:C
- added C18: 47u, Capacitor_SMD:C_1210_3225Metric_Pad1.42x2.65mm_HandSolder, symbol Device:C
- added J1: Conn_Coaxial, Connector_Coaxial:SMA_Amphenol_132203-12_Horizontal, symbol Connector:Conn_Coaxial
- added JP1, JP2: SolderJumper_2_Bridged, Jumper:SolderJumper-2_P1.3mm_Bridged_RoundedPad1.0x1.5mm, symbol Jumper:SolderJumper_2_Bridged
- added R19, R20: 50R, Resistor_SMD:R_0805_2012Metric_Pad1.15x1.40mm_HandSolder, symbol Device:R
- added R21, R22: opt, Resistor_SMD:R_0805_2012Metric_Pad1.15x1.40mm_HandSolder, symbol Device:R
- added U3: LT1469, Package_SO:SOIC-8_3.9x4.9mm_P1.27mm, symbol STM_Custom_Lib:LT1469
- added U4: LTC2326-16, Package_SO:MSOP-16_3x4.039mm_P0.5mm, symbol STM_Custom_Lib:LTC2326-16
Connections:
- net labels added: +15V, +3.3V, +5VA, -15V, GND
- wire segments 0 -> 113

Commit message: Many changes. I lost track of them...
Parts:
- removed J1: Conn_Coaxial, Connector_Coaxial:SMA_Amphenol_132203-12_Horizontal, symbol Connector:Conn_Coaxial
Changed lines of the file:
@@
 EESchema Schematic File Version 4
-LIBS:Mainboard-cache
 EELAYER 30 0
 EELAYER END
 $Descr A4 11693 8268
 encoding utf-8
-Sheet 2 3
+Sheet 2 9
 Title ""
 Date ""
@@
 	1    0    0    -1
 $EndComp
-$Comp
-L Connector:Conn_Coaxial J1
-U 1 1 5D6A7FCD
-P 2750 3100
-F 0 "J1" H 2678 3338 50  0000 C CNN
-F 1 "Conn_Coaxial" H 2678 3247 50  0000 C CNN
-F 2 "Connector_Coaxial:SMA_Amphenol_132203-12_Horizontal" H 2750 3100 50  0001 C CNN
-F 3 " ~" H 2750 3100 50  0001 C CNN
-	1    2750 3100
-	-1   0    0    -1
-$EndComp
-Wire Wire Line
+Wire Wire Line

Commit message: ADC Schematic
Parts:
- removed C10, C19, C21, C22, C24, C9: 100n, Capacitor_SMD:C_0805_2012Metric_Pad1.15x1.40mm_HandSolder, symbol Device:C
- removed C11, C12, C20, C23, C25: 10u, Capacitor_SMD:C_1206_3216Metric_Pad1.42x1.75mm_HandSolder, symbol Device:C
- removed C13, C14: 66n, Capacitor_SMD:C_0805_2012Metric_Pad1.15x1.40mm_HandSolder, symbol Device:C
- removed C15, C16, C17: opt, Capacitor_SMD:C_0805_2012Metric_Pad1.15x1.40mm_HandSolder, symbol Device:C
- removed JP1, JP2: SolderJumper_2_Bridged, Jumper:SolderJumper-2_P1.3mm_Bridged_RoundedPad1.0x1.5mm, symbol Jumper:SolderJumper_2_Bridged
- removed U4: LTC2326-16, Package_SO:MSOP-16_3x4.039mm_P0.5mm, symbol STM_Custom_Lib:LTC2326-16
- added C? (x6): 100n, Capacitor_SMD:C_0603_1608Metric_Pad1.05x0.95mm_HandSolder, symbol Device:C
- added C? (x5): 10u, Capacitor_SMD:C_0805_2012Metric_Pad1.15x1.40mm_HandSolder, symbol Device:C
- added C? (x2): 66n, Capacitor_SMD:C_0603_1608Metric_Pad1.05x0.95mm_HandSolder, symbol Device:C
- added C? (x3): opt, Capacitor_SMD:C_0603_1608Metric_Pad1.05x0.95mm_HandSolder, symbol Device:C
- added JP? (x2): Jumper, Connector_PinHeader_2.54mm:PinHeader_1x02_P2.54mm_Vertical, symbol Device:Jumper
- added U4: LTC2338-18, Package_SO:MSOP-16_3x4.039mm_P0.5mm, symbol STM_Custom_Lib:LTC2338-18
Connections:
- net labels added: +3V3, +5V, IN+, IN-
- net labels removed: +3.3V, +5VA
- wire segments 113 -> 109
Other:
- moved on the sheet: U3C

Commit message: Reference schematic
Parts:
- removed C?: 100n, Capacitor_SMD:C_0603_1608Metric_Pad1.05x0.95mm_HandSolder, symbol Device:C
- removed JP? (x2): Jumper, Connector_PinHeader_2.54mm:PinHeader_1x02_P2.54mm_Vertical, symbol Device:Jumper
- added C21: 2u2, Capacitor_SMD:C_0805_2012Metric_Pad1.15x1.40mm_HandSolder, symbol Device:C
- added JP1, JP2: Jumper, Connector_PinHeader_2.54mm:PinHeader_1x02_P2.54mm_Vertical, symbol Device:Jumper
- added U19: ADP7142AUJZ-5.0, Package_TO_SOT_SMD:TSOT-23-5, symbol Regulator_Linear:ADP7142AUJZ-5.0
- C20: renamed from C?; value 10u -> 2u2
- R21, R22: value opt -> 0R
- gave numbers to parts that had none: 14
Connections:
- net labels added: BUSY, CONV, MISO, MOSI, SCLK
- wire segments 109 -> 118
Other:
- moved on the sheet: C10, C20, C22, C23, C24, C25, C9, R19, R20

Commit message: Reference layout finished
Parts:
- added TP1: TestPoint, TestPoint:TestPoint_Pad_D1.5mm, symbol Connector:TestPoint
Connections:
- net +5V: now also TP1.1
Changed lines of the file:
@@
 Wire Wire Line
 	3400 4500 3100 4500
+$Comp
+L Connector:TestPoint TP1
+U 1 1 5ED571C5
+P 7450 1200
+F 0 "TP1" H 7508 1318 50  0000 L CNN
+F 1 "TestPoint" H 7508 1227 50  0000 L CNN
+F 2 "TestPoint:TestPoint_Pad_D1.5mm" H 7650 1200 50  0001 C CNN
+F 3 "~" H 7650 1200 50  0001 C CNN
+	1    7450 1200
+	1    0    0    -1
+$EndComp
+Wire Wire Line
+	7450 1350 7450 1200
 $EndSCHEMATC

Commit message: Mainboard layout and schematic done
Parts:
- removed JP1, JP2: Jumper, Connector_PinHeader_2.54mm:PinHeader_1x02_P2.54mm_Vertical, symbol Device:Jumper
- added C140: 1n, Capacitor_SMD:C_0603_1608Metric_Pad1.05x0.95mm_HandSolder, symbol Device:C
- added C141: 680p, Capacitor_SMD:C_0603_1608Metric_Pad1.05x0.95mm_HandSolder, symbol Device:C
- added R31, R32: 1k, Resistor_SMD:R_0603_1608Metric_Pad1.05x0.95mm_HandSolder, symbol Device:R
- added TP14: TestPoint, TestPoint:TestPoint_Pad_D1.5mm, symbol Connector:TestPoint
- C10: value 66n -> 680p; LCSC (none) -> C1630
- C11, C12, C23, C25: LCSC (none) -> C15850
- C13, C14, C19, C22, C24: LCSC (none) -> C14663
- C20, C21: LCSC (none) -> C49217
- C9: value 66n -> 1n; LCSC (none) -> C1588
- R19, R20: value 50R -> 560R; footprint Resistor_SMD:R_0805_2012Metric_Pad1.15x1.40mm_HandSolder -> Resistor_SMD:R_0603_1608Metric_Pad1.05x0.95mm_HandSolder; LCSC (none) -> C23204
- R21, R22: footprint Resistor_SMD:R_0805_2012Metric_Pad1.15x1.40mm_HandSolder -> Resistor_SMD:R_0805_2012Metric; LCSC (none) -> C17477
Connections:
- net +15V: now also TP14.1
- net GND: now also C141.2; no longer C9.2
- net at R21.2, U3.1, U3.2 (-): now also C9.1
- net at U3.3 (+): now also C10.1, R31.1
- net at U3.5 (+): now also C141.1, R32.1
- net at R22.2, U3.6 (-), U3.7: now also C140.1
- net at R19.1: now also C9.2, R31.2; no longer C9.1
- net at R20.1: now also C140.2, R32.2; no longer C10.1
Other:
- note added: "Second order bessel filters tuned to a cutoff freq. of 200 kHz"
- moved on the sheet: C11, C12, C13, C14, C22, C23, U3C

Commit message: Added images
Parts:
- C18: Reichelt (none) -> KEM X5R1210 47U
- U19: Digikey (none) -> ADP7142AUJZ-5.0-R7CT-ND
- U3: Digikey (none) -> LT1469CS8#PBF-ND
- U4: Digikey LTC2338CMS-18#PBF-ND -> LTC2338CMS-18#PBF-ND
Changed lines of the file:
@@
 F 2 "Package_SO:SOIC-8_3.9x4.9mm_P1.27mm" H 4500 3000 50  0001 C CNN
 F 3 "http://www.ti.com/lit/ds/symlink/lm358.pdf" H 4500 3000 50  0001 C CNN
+F 4 "LT1469CS8#PBF-ND " H 4500 3000 50  0001 C CNN "Digikey"
 	1    4500 3000
 	1    0    0    1
@@
 F 2 "Package_SO:SOIC-8_3.9x4.9mm_P1.27mm" H 4500 4400 50  0001 C CNN
 F 3 "http://www.ti.com/lit/ds/symlink/lm358.pdf" H 4500 4400 50  0001 C CNN
+F 4 "LT1469CS8#PBF-ND " H 4500 4400 50  0001 C CNN "Digikey"
 	2    4500 4400
 	1    0    0    1
@@
 F 2 "Package_SO:SOIC-8_3.9x4.9mm_P1.27mm" H 10550 5500 50  0001 C CNN
 F 3 "http://www.ti.com/lit/ds/symlink/lm358.pdf" H 10550 5500 50  0001 C CNN
+F 4 "LT1469CS8#PBF-ND " H 10550 5500 50  0001 C CNN "Digikey"
 	3    10550 5500
 	1    0    0    -1
@@
 F 2 "Capacitor_SMD:C_1210_3225Metric_Pad1.42x2.65mm_HandSolder" H 7088 4400 50  0001 C CNN
 F 3 "~" H 7050 4550 50  0001 C CNN
+F 4 "KEM X5R1210 47U" H 7050 4550 50  0001 C CNN "Reichelt"
 	1    7050 4550
 	1    0    0    -1
@@
 F 2 "Package_TO_SOT_SMD:TSOT-23-5" H 6650 1050 50  0001 C CIN
 F 3 "https://www.analog.com/media/en/technical-documentation/data-sheets/ADP7142.pdf" H 6650 950 50  0001 C CNN
+F 4 "ADP7142AUJZ-5.0-R7CT-ND" H 6650 1450 50  0001 C CNN "Digikey"
 	1    6650 1450
 	1    0    0    -1
@@
 F 2 "Package_SO:MSOP-16_3x4.039mm_P0.5mm" H 7550 3700 50  0001 C CIN
 F 3 "https://www.analog.com/media/en/technical-documentation/data-sheets/233818fa.pdf" H 7550 3700 50  0001 C CNN
-F 4 "LTC2338CMS-18#PBF-ND" H 7600 3700 50  0001 C CNN "Digikey"
+F 4 "LTC2338CMS-18#PBF-ND " H 7600 3700 50  0001 C CNN "Digikey"
 	1    7600 3700
 	1    0    0    -1
