File: Electronics/Mainboard/Reference.sch (KiCad schematic (older format))
At the start: 0 parts

Commit message: Reference schematic
Parts:
- added C106, C109, C113, C114, C118, C119: 10u, Capacitor_SMD:C_0805_2012Metric_Pad1.15x1.40mm_HandSolder, symbol Device:C
- added C107, C108, C111, C112, C116, C117: 100n, Capacitor_SMD:C_0805_2012Metric_Pad1.15x1.40mm_HandSolder, symbol Device:C
- added C110, C115: opt, Capacitor_SMD:C_0805_2012Metric_Pad1.15x1.40mm_HandSolder, symbol Device:C
- added J5: Conn_Coaxial, Connector_Coaxial:SMB_Jack_Vertical, symbol Connector:Conn_Coaxial
- added R23: 1k5, Capacitor_SMD:C_0805_2012Metric_Pad1.15x1.40mm_HandSolder, symbol Device:R
- added R24, R25, R26, R27, R28: 1k, Capacitor_SMD:C_0805_2012Metric_Pad1.15x1.40mm_HandSolder, symbol Device:R
- added TP2, TP3, TP4, TP5: TestPoint, TestPoint:TestPoint_Loop_D1.80mm_Drill1.0mm_Beaded, symbol Connector:TestPoint
- added U20: ADR4550, Package_SO:SOIC-8_3.9x4.9mm_P1.27mm, symbol Reference_Voltage:ADR4550
- added U21: AD8676, Package_SO:SOIC-8_3.9x4.9mm_P1.27mm, symbol STM_Custom_Lib:AD8676
- added U22: AD8675, Package_SO:SOIC-8_3.9x4.9mm_P1.27mm, symbol STM_Custom_Lib:AD8675
Connections:
- net +15V: now also C106.1, C107.1, C111.1, C113.1, C116.1, C118.1, U20.2 (IN), U21.8 (V+), U22.7 (V+)
- net -15V: now also C112.2, C114.2, C117.2, C119.2, U21.4 (V-), U22.4 (V-)
- net GND: now also C106.2, C107.2, C108.2, C109.2, C111.2, C112.1, C113.2, C114.1, C116.2, C117.1, C118.2, C119.1, J5.2 (Ext), R24.2, U20.4 (GND), U21.5 (+)
- net REF_N: now also C115.2, R28.1, TP5.1, U21.7
- net REF_P: now also C110.2, R26.1, TP4.1, U22.6
- new net: C110.1, R24.1, R26.2, U22.2 (-)
- new net: C109.1, J5.1 (In), R23.1, U21.3 (+), U22.3 (+)
- new net: R25.2, TP3.1, U21.1, U21.2 (-)
- new net: C115.1, R25.1, R27.2, U21.6 (-)
- new net: C108.1, R23.2, TP2.1, U20.6 (OUT)
- new net: R27.1, R28.2
Other:
- note added: "Pin compatible references:\nADR435\nADR445"

Commit message: Layout progress
Parts:
- removed J5: Conn_Coaxial, Connector_Coaxial:SMB_Jack_Vertical, symbol Connector:Conn_Coaxial
- added TP6: TestPoint, TestPoint:TestPoint_Loop_D1.80mm_Drill1.0mm_Beaded, symbol Connector:TestPoint
Connections:
- net at C109.1, R23.1, U21.3 (+)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: now also TP6.1
Changed lines of the file:
@@
 	6100 2400 6100 2300
-$Comp
-L Connector:Conn_Coaxial J5
-U 1 1 5F1A47C7
-P 4050 2450
-F 0 "J5" H 4150 2425 50  0000 L CNN
-F 1 "Conn_Coaxial" H 4150 2334 50  0000 L CNN
-F 2 "Connector_Coaxial:SMB_Jack_Vertical" H 4050 2450 50  0001 C CNN
-F 3 " ~" H 4050 2450 50  0001 C CNN
-	1    4050 2450
-	1    0    0    -1
-$EndComp
 $Comp
 L Reference_Voltage:ADR4550 U20
@@
 	3600 3200 2900 3200
 Connection ~ 2900 3200
-Wire Wire Line
-	3600 2800 3800 2800
 Connection ~ 3600 2800
-Wire Wire Line
-	3850 2450 3800 2450
-Wire Wire Line
-	3800 2450 3800 2800
-Wire Wire Line
-	3600 3200 4050 3200
-Wire Wire Line
-	4050 3200 4050 2650
-Connection ~ 3600 3200
-Connection ~ 3800 2800
 $Comp
 L Device:R R?
@@
 Connection ~ 7100 3650
 Wire Wire Line
-	3800 2800 4800 2800
-Wire Wire Line
 	4800 2800 4800 3850
 Connection ~ 4800 2800
@@
 Text Notes 2350 2250 0    50   ~ 0
 Pin compatible references:\nADR435\nADR445
+Wire Wire Line
+	3600 2800 4800 2800
+$Comp
+L Connector:TestPoint TP6
+U 1 1 5F2E4DA1
+P 3600 2700
+F 0 "TP6" H 3658 2818 50  0001 L CNN
+F 1 "TestPoint" H 3658 2727 50  0001 L CNN
+F 2 "TestPoint:TestPoint_Loop_D1.80mm_Drill1.0mm_Beaded" H 3800 2700 50  0001 C CNN
+F 3 "~" H 3800 2700 50  0001 C CNN
+	1    3600 2700
+	1    0    0    -1
+$EndComp
+Wire Wire Line
+	3600 2700 3600 2800
 $EndSCHEMATC

Commit message: Layout nearly finished
Parts:
- TP4, TP5: footprint TestPoint:TestPoint_Loop_D1.80mm_Drill1.0mm_Beaded -> TestPoint:TestPoint_Pad_D2.0mm
Changed lines of the file:
@@
 F 0 "TP4" H 7308 2718 50  0001 L CNN
 F 1 "TestPoint" H 7308 2627 50  0001 L CNN
-F 2 "TestPoint:TestPoint_Loop_D1.80mm_Drill1.0mm_Beaded" H 7450 2600 50  0001 C CNN
+F 2 "TestPoint:TestPoint_Pad_D2.0mm" H 7450 2600 50  0001 C CNN
 F 3 "~" H 7450 2600 50  0001 C CNN
 	1    7250 2600
@@
 F 0 "TP5" H 7308 4068 50  0001 L CNN
 F 1 "TestPoint" H 7308 3977 50  0001 L CNN
-F 2 "TestPoint:TestPoint_Loop_D1.80mm_Drill1.0mm_Beaded" H 7450 3950 50  0001 C CNN
+F 2 "TestPoint:TestPoint_Pad_D2.0mm" H 7450 3950 50  0001 C CNN
 F 3 "~" H 7450 3950 50  0001 C CNN
 	1    7250 3950

Commit message: Mainboard layout and schematic done
Parts:
- C106, C109, C113, C114, C118, C119: LCSC (none) -> C15850
- C107, C108, C111, C112, C116, C117: footprint Capacitor_SMD:C_0805_2012Metric_Pad1.15x1.40mm_HandSolder -> Capacitor_SMD:C_0603_1608Metric_Pad1.05x0.95mm_HandSolder; LCSC (none) -> C14663
- R23: value 1k5 -> 1k; footprint Capacitor_SMD:C_0805_2012Metric_Pad1.15x1.40mm_HandSolder -> Resistor_SMD:R_0805_2012Metric; LCSC (none) -> C17513
- R24, R25, R26, R27, R28: footprint Capacitor_SMD:C_0805_2012Metric_Pad1.15x1.40mm_HandSolder -> Resistor_SMD:R_0805_2012Metric; LCSC (none) -> C17513
Other:
- note added: "+10V Reference Output"
- note added: "-10V Reference Output"
- note added: "5V Reference Output"
Changed lines of the file:
@@
 F 2 "Package_SO:SOIC-8_3.9x4.9mm_P1.27mm" H 5200 3950 50  0001 C CNN
 F 3 "https://www.digikey.de/product-detail/de/analog-devices-inc/AD8676ARZ/AD8676ARZ-ND/1246063" H 5200 3950 50  0001 C CNN
+F 4 "" H 5200 3950 50  0001 C CNN "LCSC"
 	1    5200 3950
 	1    0    0    -1
@@
 F 2 "Package_SO:SOIC-8_3.9x4.9mm_P1.27mm" H 6550 4050 50  0001 C CNN
 F 3 "https://www.digikey.de/product-detail/de/analog-devices-inc/AD8676ARZ/AD8676ARZ-ND/1246063" H 6550 4050 50  0001 C CNN
+F 4 "" H 6550 4050 50  0001 C CNN "LCSC"
 	2    6550 4050
 	1    0    0    1
@@
 AR Path="/5EE4ADA7/5F198A86" Ref="R23"  Part="1"
 F 0 "R23" V 3200 2700 50  0000 C CNN
-F 1 "1k5" V 3200 2900 50  0000 C CNN
-F 2 "Capacitor_SMD:C_0805_2012Metric_Pad1.15x1.40mm_HandSolder" V 3230 2800 50  0001 C CNN
+F 1 "1k" V 3200 2900 50  0000 C CNN
+F 2 "Resistor_SMD:R_0805_2012Metric" V 3230 2800 50  0001 C CNN
 F 3 "~" H 3300 2800 50  0001 C CNN
+F 4 "C17513" H 3300 2800 50  0001 C CNN "LCSC"
 	1    3300 2800
 	0    1    1    0
@@
 F 2 "Capacitor_SMD:C_0805_2012Metric_Pad1.15x1.40mm_HandSolder" H 1788 2650 50  0001 C CNN
 F 3 "~" H 1750 2800 50  0001 C CNN
+F 4 "C15850" H 1750 2800 50  0001 C CNN "LCSC"
 	1    1750 2800
 	1    0    0    -1
@@
 F 0 "C108" H 2950 3100 50  0000 L CNN
 F 1 "100n" H 3150 2900 50  0000 R CNN
-F 2 "Capacitor_SMD:C_0805_2012Metric_Pad1.15x1.40mm_HandSolder" H 2938 2850 50  0001 C CNN
+F 2 "Capacitor_SMD:C_0603_1608Metric_Pad1.05x0.95mm_HandSolder" H 2938 2850 50  0001 C CNN
 F 3 "~" H 2900 3000 50  0001 C CNN
+F 4 "C14663" H 2900 3000 50  0001 C CNN "LCSC"
 	1    2900 3000
 	1    0    0    -1
@@
 F 2 "Capacitor_SMD:C_0805_2012Metric_Pad1.15x1.40mm_HandSolder" H 3638 2850 50  0001 C CNN
 F 3 "~" H 3600 3000 50  0001 C CNN
+F 4 "C15850" H 3600 3000 50  0001 C CNN "LCSC"
 	1    3600 3000
 	1    0    0    -1
@@
 F 0 "R24" V 5450 2500 50  0000 C CNN
 F 1 "1k" V 5450 2700 50  0000 C CNN
-F 2 "Capacitor_SMD:C_0805_2012Metric_Pad1.15x1.40mm_HandSolder" V 5480 2600 50  0001 C CNN
+F 2 "Resistor_SMD:R_0805_2012Metric" V 5480 2600 50  0001 C CNN
 F 3 "~" H 5550 2600 50  0001 C CNN
+F 4 "C17513" H 5550 2600 50  0001 C CNN "LCSC"
 	1    5550 2600
 	0    1    1    0
@@
 F 0 "R26" V 6100 2050 50  0000 C CNN
 F 1 "1k" V 6100 2250 50  0000 C CNN
-F 2 "Capacitor_SMD:C_0805_2012Metric_Pad1.15x1.40mm_HandSolder" V 6130 2150 50  0001 C CNN
+F 2 "Resistor_SMD:R_0805_2012Metric" V 6130 2150 50  0001 C CNN
 F 3 "~" H 6200 2150 50  0001 C CNN
+F 4 "C17513" H 6200 2150 50  0001 C CNN "LCSC"
 	1    6200 2150
 	0    1    1    0
@@
 F 0 "R25" V 5800 3850 50  0000 C CNN
 F 1 "1k" V 5800 4050 50  0000 C CNN
-F 2 "Capacitor_SMD:C_0805_2012Metric_Pad1.15x1.40mm_HandSolder" V 5830 3950 50  0001 C CNN
+F 2 "Resistor_SMD:R_0805_2012Metric" V 5830 3950 50  0001 C CNN
 F 3 "~" H 5900 3950 50  0001 C CNN
+F 4 "C17513" H 5900 3950 50  0001 C CNN "LCSC"
 	1    5900 3950
 	0    1    1    0
@@
 F 0 "R27" V 6350 3550 50  0000 C CNN
 F 1 "1k" V 6350 3750 50  0000 C CNN
-F 2 "Capacitor_SMD:C_0805_2012Metric_Pad1.15x1.40mm_HandSolder" V 6380 3650 50  0001 C CNN
+F 2 "Resistor_SMD:R_0805_2012Metric" V 6380 3650 50  0001 C CNN
 F 3 "~" H 6450 3650 50  0001 C CNN
+F 4 "C17513" H 6450 3650 50  0001 C CNN "LCSC"
 	1    6450 3650
 	0    1    1    0
@@
 F 0 "R28" V 6750 3550 50  0000 C CNN
 F 1 "1k" V 6750 3750 50  0000 C CNN
-F 2 "Capacitor_SMD:C_0805_2012Metric_Pad1.15x1.40mm_HandSolder" V 6780 3650 50  0001 C CNN
+F 2 "Resistor_SMD:R_0805_2012Metric" V 6780 3650 50  0001 C CNN
 F 3 "~" H 6850 3650 50  0001 C CNN
+F 4 "C17513" H 6850 3650 50  0001 C CNN "LCSC"
 	1    6850 3650
 	0    1    1    0
@@
 F 0 "C107" H 2050 2900 50  0000 L CNN
 F 1 "100n" H 2250 2700 50  0000 R CNN
-F 2 "Capacitor_SMD:C_0805_2012Metric_Pad1.15x1.40mm_HandSolder" H 2038 2650 50  0001 C CNN
+F 2 "Capacitor_SMD:C_0603_1608Metric_Pad1.05x0.95mm_HandSolder" H 2038 2650 50  0001 C CNN
 F 3 "~" H 2000 2800 50  0001 C CNN
+F 4 "C14663" H 2000 2800 50  0001 C CNN "LCSC"
 	1    2000 2800
 	1    0    0    -1
@@
 F 2 "Package_SO:SOIC-8_3.9x4.9mm_P1.27mm" H 7400 5250 50  0001 C CNN
 F 3 "https://www.digikey.de/product-detail/de/analog-devices-inc/AD8676ARZ/AD8676ARZ-ND/1246063" H 7400 5250 50  0001 C CNN
+F 4 "" H 7400 5250 50  0001 C CNN "LCSC"
 	3    7400 5250
 	1    0    0    -1
@@
 F 2 "Capacitor_SMD:C_0805_2012Metric_Pad1.15x1.40mm_HandSolder" H 6988 4850 50  0001 C CNN
 F 3 "~" H 6950 5000 50  0001 C CNN
+F 4 "C15850" H 6950 5000 50  0001 C CNN "LCSC"
 	1    6950 5000
 	1    0    0    -1
@@
 F 2 "Capacitor_SMD:C_0805_2012Metric_Pad1.15x1.40mm_HandSolder" H 6988 5450 50  0001 C CNN
 F 3 "~" H 6950 5600 50  0001 C CNN
+F 4 "C15850" H 6950 5600 50  0001 C CNN "LCSC"
 	1    6950 5600
 	1    0    0    -1
@@
 F 2 "Capacitor_SMD:C_0805_2012Metric_Pad1.15x1.40mm_HandSolder" H 6488 4850 50  0001 C CNN
 F 3 "~" H 6450 5000 50  0001 C CNN
+F 4 "C15850" H 6450 5000 50  0001 C CNN "LCSC"
 	1    6450 5000
 	1    0    0    -1
@@
 F 0 "C111" V 6300 5050 50  0000 L CNN
 F 1 "100n" V 6300 4950 50  0000 R CNN
-F 2 "Capacitor_SMD:C_0805_2012Metric_Pad1.15x1.40mm_HandSolder" H 6238 4850 50  0001 C CNN
+F 2 "Capacitor_SMD:C_0603_1608Metric_Pad1.05x0.95mm_HandSolder" H 6238 4850 50  0001 C CNN
 F 3 "~" H 6200 5000 50  0001 C CNN
+F 4 "C14663" H 6200 5000 50  0001 C CNN "LCSC"
 	1    6200 5000
 	1    0    0    -1
@@
 F 2 "Capacitor_SMD:C_0805_2012Metric_Pad1.15x1.40mm_HandSolder" H 6488 5450 50  0001 C CNN
 F 3 "~" H 6450 5600 50  0001 C CNN
+F 4 "C15850" H 6450 5600 50  0001 C CNN "LCSC"
 	1    6450 5600
 	1    0    0    -1
@@
 F 0 "C112" V 6300 5650 50  0000 L CNN
 F 1 "100n" V 6300 5550 50  0000 R CNN
-F 2 "Capacitor_SMD:C_0805_2012Metric_Pad1.15x1.40mm_HandSolder" H 6238 5450 50  0001 C CNN
+F 2 "Capacitor_SMD:C_0603_1608Metric_Pad1.05x0.95mm_HandSolder" H 6238 5450 50  0001 C CNN
 F 3 "~" H 6200 5600 50  0001 C CNN
+F 4 "C14663" H 6200 5600 50  0001 C CNN "LCSC"
 	1    6200 5600
 	1    0    0    -1
@@
 F 0 "C117" V 6800 5650 50  0000 L CNN
 F 1 "100n" V 6800 5550 50  0000 R CNN
-F 2 "Capacitor_SMD:C_0805_2012Metric_Pad1.15x1.40mm_HandSolder" H 6738 5450 50  0001 C CNN
+F 2 "Capacitor_SMD:C_0603_1608Metric_Pad1.05x0.95mm_HandSolder" H 6738 5450 50  0001 C CNN
 F 3 "~" H 6700 5600 50  0001 C CNN
+F 4 "C14663" H 6700 5600 50  0001 C CNN "LCSC"
 	1    6700 5600
 	1    0    0    -1
@@
 F 0 "C116" V 6800 5050 50  0000 L CNN
 F 1 "100n" V 6800 4950 50  0000 R CNN
-F 2 "Capacitor_SMD:C_0805_2012Metric_Pad1.15x1.40mm_HandSolder" H 6738 4850 50  0001 C CNN
+F 2 "Capacitor_SMD:C_0603_1608Metric_Pad1.05x0.95mm_HandSolder" H 6738 4850 50  0001 C CNN
 F 3 "~" H 6700 5000 50  0001 C CNN
+F 4 "C14663" H 6700 5000 50  0001 C CNN "LCSC"
 	1    6700 5000
 	1    0    0    -1
@@
 Wire Wire Line
 	3600 2700 3600 2800
+Text Notes 3950 2700 0    50   ~ 0
+5V Reference Output
+Text Notes 7400 2950 0    50   ~ 0
++10V Reference Output
+Text Notes 7400 4300 0    50   ~ 0
+-10V Reference Output
 $EndSCHEMATC

Commit message: Added images
Parts:
- U20: Digikey (none) -> ADR4550ARZ-ND
- U21: Digikey (none) -> AD8676ARZ-ND
- U22: Digikey (none) -> AD8675ARZ-REEL7CT-ND
Changed lines of the file:
@@
 F 2 "Package_SO:SOIC-8_3.9x4.9mm_P1.27mm" H 6400 2950 50  0001 C CNN
 F 3 "" H 6400 2950 50  0001 C CNN
+F 4 "AD8675ARZ-REEL7CT-ND " H 6200 2700 50  0001 C CNN "Digikey"
 	1    6200 2700
 	1    0    0    -1
@@
 F 3 "https://www.digikey.de/product-detail/de/analog-devices-inc/AD8676ARZ/AD8676ARZ-ND/1246063" H 5200 3950 50  0001 C CNN
 F 4 "" H 5200 3950 50  0001 C CNN "LCSC"
+F 5 "AD8676ARZ-ND" H 5200 3950 50  0001 C CNN "Digikey"
 	1    5200 3950
 	1    0    0    -1
@@
 F 3 "https://www.digikey.de/product-detail/de/analog-devices-inc/AD8676ARZ/AD8676ARZ-ND/1246063" H 6550 4050 50  0001 C CNN
 F 4 "" H 6550 4050 50  0001 C CNN "LCSC"
+F 5 "AD8676ARZ-ND" H 6550 4050 50  0001 C CNN "Digikey"
 	2    6550 4050
 	1    0    0    1
@@
 F 2 "Package_SO:SOIC-8_3.9x4.9mm_P1.27mm" H 2550 2500 50  0001 C CIN
 F 3 "https://www.analog.com/media/en/technical-documentation/data-sheets/ADR4520_4525_4530_4533_4540_4550.pdf" H 2550 2450 50  0001 C CIN
+F 4 "ADR4550ARZ-ND" H 2450 2800 50  0001 C CNN "Digikey"
 	1    2450 2800
 	1    0    0    -1
@@
 F 3 "https://www.digikey.de/product-detail/de/analog-devices-inc/AD8676ARZ/AD8676ARZ-ND/1246063" H 7400 5250 50  0001 C CNN
 F 4 "" H 7400 5250 50  0001 C CNN "LCSC"
+F 5 "AD8676ARZ-ND" H 7400 5250 50  0001 C CNN "Digikey"
 	3    7400 5250
 	1    0    0    -1
