File: Electronics/Mainboard/Single-DAC.sch (KiCad schematic (older format))
At the start: 20 parts, among them U10 AD8675, U5 AD5781, U9 AD8676xR

Commit message: Layout of piezo DACs ready
Parts:
- removed C33, C38, C41, C42, C45, C46: 100n, Capacitor_SMD:C_0805_2012Metric_Pad1.15x1.40mm_HandSolder, symbol Device:C
- removed C34: 10u, Capacitor_SMD:C_0805_2012Metric_Pad1.15x1.40mm_HandSolder, symbol Device:C
- added C26, C29, C30, C31, C32: 100n, Capacitor_SMD:C_0603_1608Metric_Pad1.05x0.95mm_HandSolder, symbol Device:C
- added C71, C72: 10p, Capacitor_SMD:C_0603_1608Metric_Pad1.05x0.95mm_HandSolder, symbol Device:C
- added JP5: Jumper, Connector_PinHeader_2.54mm:PinHeader_1x02_P2.54mm_Vertical, symbol Device:Jumper
- C27, C37: footprint Capacitor_SMD:C_0805_2012Metric_Pad1.15x1.40mm_HandSolder -> Capacitor_SMD:C_0603_1608Metric_Pad1.05x0.95mm_HandSolder
Connections:
- net labels added: 3V3, GND, ~CS, ~LDAC
- net labels removed: !CLR, !LDAC, !RST, !SYNC, +3.3V, GNDA, GNDD
- wire segments 102 -> 106

Commit message: ADC Schematic
Changed lines of the file:
@@
 AR Path="/5EE5BDE4/5F11C2AA/5DA35D26" Ref="U?"  Part="1"
 AR Path="/5F11EDFC/5DA35D26" Ref="U16"  Part="1"
-F 0 "U16" H 5100 3850 50  0000 L CNN
+F 0 "U8" H 5100 3850 50  0000 L CNN
 F 1 "AD5781" H 5000 3750 50  0000 L CNN
 F 2 "Package_SO:TSSOP-20_4.4x6.5mm_P0.65mm" H 4550 3800 50  0001 C CNN
@@
 AR Path="/5EE5BDE4/5F11C2AA/5DA6205A" Ref="C?"  Part="1"
 AR Path="/5F11EDFC/5DA6205A" Ref="C91"  Part="1"
-F 0 "C91" H 6315 3546 50  0000 L CNN
+F 0 "C28" H 6315 3546 50  0000 L CNN
 F 1 "10p" H 6315 3455 50  0000 L CNN
 F 2 "Capacitor_SMD:C_0603_1608Metric_Pad1.05x0.95mm_HandSolder" H 6238 3350 50  0001 C CNN
@@
 AR Path="/5EE5BDE4/5F11C2AA/5DAF59CE" Ref="C?"  Part="1"
 AR Path="/5F11EDFC/5DAF59CE" Ref="C102"  Part="1"
-F 0 "C102" V 9450 4150 50  0000 L CNN
+F 0 "C47" V 9450 4150 50  0000 L CNN
 F 1 "10u" V 9450 4050 50  0000 R CNN
 F 2 "Capacitor_SMD:C_0805_2012Metric_Pad1.15x1.40mm_HandSolder" H 9388 3950 50  0001 C CNN
@@
 AR Path="/5EE5BDE4/5F11C2AA/5DAFF8A7" Ref="C?"  Part="1"
 AR Path="/5F11EDFC/5DAFF8A7" Ref="C94"  Part="1"
-F 0 "C94" V 8550 2150 50  0000 L CNN
+F 0 "C52" V 8550 2150 50  0000 L CNN
 F 1 "100n" V 8550 2050 50  0000 R CNN
 F 2 "Capacitor_SMD:C_0603_1608Metric_Pad1.05x0.95mm_HandSolder" H 8488 1950 50  0001 C CNN
@@
 AR Path="/5EE5BDE4/5F11C2AA/5DAFF8B1" Ref="C?"  Part="1"
 AR Path="/5F11EDFC/5DAFF8B1" Ref="C92"  Part="1"
-F 0 "C92" V 8300 2150 50  0000 L CNN
+F 0 "C50" V 8300 2150 50  0000 L CNN
 F 1 "10u" V 8300 2050 50  0000 R CNN
 F 2 "Capacitor_SMD:C_0805_2012Metric_Pad1.15x1.40mm_HandSolder" H 8238 1950 50  0001 C CNN
@@
 AR Path="/5EE5BDE4/5F11C2AA/5DB37044" Ref="C?"  Part="1"
 AR Path="/5F11EDFC/5DB37044" Ref="C93"  Part="1"
-F 0 "C93" V 8300 2650 50  0000 L CNN
+F 0 "C51" V 8300 2650 50  0000 L CNN
 F 1 "10u" V 8300 2550 50  0000 R CNN
 F 2 "Capacitor_SMD:C_0805_2012Metric_Pad1.15x1.40mm_HandSolder" H 8238 2450 50  0001 C CNN
@@
 AR Path="/5EE5BDE4/5F11C2AA/5DB4EB12" Ref="C?"  Part="1"
 AR Path="/5F11EDFC/5DB4EB12" Ref="C96"  Part="1"
-F 0 "C96" V 8800 2150 50  0000 L CNN
+F 0 "C54" V 8800 2150 50  0000 L CNN
 F 1 "10u" V 8800 2050 50  0000 R CNN
 F 2 "Capacitor_SMD:C_0805_2012Metric_Pad1.15x1.40mm_HandSolder" H 8738 1950 50  0001 C CNN
@@
 AR Path="/5EE5BDE4/5F11C2AA/5DB596AD" Ref="C?"  Part="1"
 AR Path="/5F11EDFC/5DB596AD" Ref="C97"  Part="1"
-F 0 "C97" V 8800 2650 50  0000 L CNN
+F 0 "C55" V 8800 2650 50  0000 L CNN
 F 1 "10u" V 8800 2550 50  0000 R CNN
 F 2 "Capacitor_SMD:C_0805_2012Metric_Pad1.15x1.40mm_HandSolder" H 8738 2450 50  0001 C CNN
@@
 AR Path="/5EE5BDE4/5F11C2AA/5DB7BE8B" Ref="C?"  Part="1"
 AR Path="/5F11EDFC/5DB7BE8B" Ref="C100"  Part="1"
-F 0 "C100" V 9300 2150 50  0000 L CNN
+F 0 "C58" V 9300 2150 50  0000 L CNN
 F 1 "10u" V 9300 2050 50  0000 R CNN
 F 2 "Capacitor_SMD:C_0805_2012Metric_Pad1.15x1.40mm_HandSolder" H 9238 1950 50  0001 C CNN
@@
 AR Path="/5EE5BDE4/5F11C2AA/5DB7BEA1" Ref="C?"  Part="1"
 AR Path="/5F11EDFC/5DB7BEA1" Ref="C101"  Part="1"
-F 0 "C101" V 9300 2650 50  0000 L CNN
+F 0 "C59" V 9300 2650 50  0000 L CNN
 F 1 "10u" V 9300 2550 50  0000 R CNN
 F 2 "Capacitor_SMD:C_0805_2012Metric_Pad1.15x1.40mm_HandSolder" H 9238 2450 50  0001 C CNN
@@
 AR Path="/5EE5BDE4/5F11C2AA/5EBF2A39" Ref="U?"  Part="1"
 AR Path="/5F11EDFC/5EBF2A39" Ref="U17"  Part="1"
-F 0 "U17" V 5304 2570 50  0000 R CNN
+F 0 "U9" V 5304 2570 50  0000 R CNN
 F 1 "AD8676xR" V 5395 2570 50  0000 R CNN
 F 2 "Package_SO:SOIC-8_3.9x4.9mm_P1.27mm" H 5450 2800 50  0001 C CNN
@@
 AR Path="/5EE5BDE4/5F11C2AA/5EBF3E04" Ref="U?"  Part="3"
 AR Path="/5F11EDFC/5EBF3E04" Ref="U17"  Part="3"
-F 0 "U17" H 9858 2396 50  0000 L CNN
+F 0 "U9" H 9858 2396 50  0000 L CNN
 F 1 "AD8676xR" H 9858 2305 50  0000 L CNN
 F 2 "Package_SO:SOIC-8_3.9x4.9mm_P1.27mm" H 9900 2350 50  0001 C CNN
@@
 AR Path="/5EE5BDE4/5F11C2AA/5EC22718" Ref="U?"  Part="1"
 AR Path="/5F11EDFC/5EC22718" Ref="U18"  Part="1"
-F 0 "U18" H 6800 3600 50  0000 L CNN
+F 0 "U10" H 6800 3600 50  0000 L CNN
 F 1 "AD8675" H 6750 3500 50  0000 L CNN
 F 2 "Package_SO:SOIC-8_3.9x4.9mm_P1.27mm" H 6950 4000 50  0001 C CNN
@@
 AR Path="/5EE5BDE4/5F11C2AA/5EE92855" Ref="C?"  Part="1"
 AR Path="/5F11EDFC/5EE92855" Ref="C95"  Part="1"
-F 0 "C95" V 8550 2650 50  0000 L CNN
+F 0 "C26" V 8550 2650 50  0000 L CNN
 F 1 "100n" V 8550 2550 50  0000 R CNN
 F 2 "Capacitor_SMD:C_0603_1608Metric_Pad1.05x0.95mm_HandSolder" H 8488 2450 50  0001 C CNN
@@
 AR Path="/5EE5BDE4/5F11C2AA/5EE92AC5" Ref="C?"  Part="1"
 AR Path="/5F11EDFC/5EE92AC5" Ref="C99"  Part="1"
-F 0 "C99" V 9050 2650 50  0000 L CNN
+F 0 "C29" V 9050 2650 50  0000 L CNN
 F 1 "100n" V 9050 2550 50  0000 R CNN
 F 2 "Capacitor_SMD:C_0603_1608Metric_Pad1.05x0.95mm_HandSolder" H 8988 2450 50  0001 C CNN
@@
 AR Path="/5EE5BDE4/5F11C2AA/5EE92D85" Ref="C?"  Part="1"
 AR Path="/5F11EDFC/5EE92D85" Ref="C98"  Part="1"
-F 0 "C98" V 9050 2150 50  0000 L CNN
+F 0 "C27" V 9050 2150 50  0000 L CNN
 F 1 "100n" V 9050 2050 50  0000 R CNN
 F 2 "Capacitor_SMD:C_0603_1608Metric_Pad1.05x0.95mm_HandSolder" H 8988 1950 50  0001 C CNN
@@
 AR Path="/5EE5BDE4/5F11C2AA/5EE931CA" Ref="C?"  Part="1"
 AR Path="/5F11EDFC/5EE931CA" Ref="C103"  Part="1"
-F 0 "C103" V 9550 2150 50  0000 L CNN
+F 0 "C30" V 9550 2150 50  0000 L CNN
 F 1 "100n" V 9550 2050 50  0000 R CNN
 F 2 "Capacitor_SMD:C_0603_1608Metric_Pad1.05x0.95mm_HandSolder" H 9488 1950 50  0001 C CNN
@@
 AR Path="/5EE5BDE4/5F11C2AA/5EE9354C" Ref="C?"  Part="1"
 AR Path="/5F11EDFC/5EE9354C" Ref="C104"  Part="1"
-F 0 "C104" V 9550 2650 50  0000 L CNN
+F 0 "C31" V 9550 2650 50  0000 L CNN
 F 1 "100n" V 9550 2550 50  0000 R CNN
 F 2 "Capacitor_SMD:C_0603_1608Metric_Pad1.05x0.95mm_HandSolder" H 9488 2450 50  0001 C CNN
@@
 AR Path="/5EE5BDE4/5F11C2AA/5EE955F2" Ref="C?"  Part="1"
 AR Path="/5F11EDFC/5EE955F2" Ref="C105"  Part="1"
-F 0 "C105" V 9700 4150 50  0000 L CNN
+F 0 "C32" V 9700 4150 50  0000 L CNN
 F 1 "100n" V 9700 4050 50  0000 R CNN
 F 2 "Capacitor_SMD:C_0603_1608Metric_Pad1.05x0.95mm_HandSolder" H 9638 3950 50  0001 C CNN
@@
 AR Path="/5EE5BDE4/5F11C2AA/5ED378D9" Ref="C?"  Part="1"
 AR Path="/5F11EDFC/5ED378D9" Ref="C89"  Part="1"
-F 0 "C89" H 4915 2346 50  0000 L CNN
+F 0 "C71" H 4915 2346 50  0000 L CNN
 F 1 "10p" H 4915 2255 50  0000 L CNN
 F 2 "Capacitor_SMD:C_0603_1608Metric_Pad1.05x0.95mm_HandSolder" H 4838 2150 50  0001 C CNN
@@
 AR Path="/5EE5BDE4/5F11C2AA/5ED4490E" Ref="C?"  Part="1"
 AR Path="/5F11EDFC/5ED4490E" Ref="C90"  Part="1"
-F 0 "C90" H 4915 5196 50  0000 L CNN
+F 0 "C72" H 4915 5196 50  0000 L CNN
 F 1 "10p" H 4915 5105 50  0000 L CNN
 F 2 "Capacitor_SMD:C_0603_1608Metric_Pad1.05x0.95mm_HandSolder" H 4838 5000 50  0001 C CNN
@@
 AR Path="/5EE5BDE4/5F11C2AA/5EBF327E" Ref="U?"  Part="2"
 AR Path="/5F11EDFC/5EBF327E" Ref="U17"  Part="2"
-F 0 "U17" V 5396 4370 50  0000 R CNN
+F 0 "U9" V 5396 4370 50  0000 R CNN
 F 1 "AD8676xR" V 5305 4370 50  0000 R CNN
 F 2 "Package_SO:SOIC-8_3.9x4.9mm_P1.27mm" H 5450 4600 50  0001 C CNN
@@
 AR Path="/5EE5BDE4/5F11C2AA/5F0961D2" Ref="JP?"  Part="1"
 AR Path="/5F11EDFC/5F0961D2" Ref="JP10"  Part="1"
-F 0 "JP10" H 7700 3923 50  0000 C CNN
+F 0 "JP5" H 7700 3923 50  0000 C CNN
 F 1 "Jumper" H 7700 3923 50  0001 C CNN
 F 2 "Connector_PinHeader_2.54mm:PinHeader_1x02_P2.54mm_Vertical" H 7700 3750 50  0001 C CNN

Commit message: Reference schematic
Changed lines of the file:
@@
 $Descr A4 11693 8268
 encoding utf-8
-Sheet 11 11
+Sheet 6 11
 Title ""
 Date ""
@@
 AR Path="/5EE5BDE4/5F11C2AA/5DA35D26" Ref="U?"  Part="1"
 AR Path="/5F11EDFC/5DA35D26" Ref="U16"  Part="1"
-F 0 "U8" H 5100 3850 50  0000 L CNN
+F 0 "U16" H 5100 3850 50  0000 L CNN
 F 1 "AD5781" H 5000 3750 50  0000 L CNN
 F 2 "Package_SO:TSSOP-20_4.4x6.5mm_P0.65mm" H 4550 3800 50  0001 C CNN
@@
 AR Path="/5EE5BDE4/5F11C2AA/5DA6205A" Ref="C?"  Part="1"
 AR Path="/5F11EDFC/5DA6205A" Ref="C91"  Part="1"
-F 0 "C28" H 6315 3546 50  0000 L CNN
+F 0 "C91" H 6315 3546 50  0000 L CNN
 F 1 "10p" H 6315 3455 50  0000 L CNN
 F 2 "Capacitor_SMD:C_0603_1608Metric_Pad1.05x0.95mm_HandSolder" H 6238 3350 50  0001 C CNN
@@
 AR Path="/5EE5BDE4/5F11C2AA/5DAF59CE" Ref="C?"  Part="1"
 AR Path="/5F11EDFC/5DAF59CE" Ref="C102"  Part="1"
-F 0 "C47" V 9450 4150 50  0000 L CNN
+F 0 "C102" V 9450 4150 50  0000 L CNN
 F 1 "10u" V 9450 4050 50  0000 R CNN
 F 2 "Capacitor_SMD:C_0805_2012Metric_Pad1.15x1.40mm_HandSolder" H 9388 3950 50  0001 C CNN
@@
 AR Path="/5EE5BDE4/5F11C2AA/5DAFF8A7" Ref="C?"  Part="1"
 AR Path="/5F11EDFC/5DAFF8A7" Ref="C94"  Part="1"
-F 0 "C52" V 8550 2150 50  0000 L CNN
+F 0 "C94" V 8550 2150 50  0000 L CNN
 F 1 "100n" V 8550 2050 50  0000 R CNN
 F 2 "Capacitor_SMD:C_0603_1608Metric_Pad1.05x0.95mm_HandSolder" H 8488 1950 50  0001 C CNN
@@
 AR Path="/5EE5BDE4/5F11C2AA/5DAFF8B1" Ref="C?"  Part="1"
 AR Path="/5F11EDFC/5DAFF8B1" Ref="C92"  Part="1"
-F 0 "C50" V 8300 2150 50  0000 L CNN
+F 0 "C92" V 8300 2150 50  0000 L CNN
 F 1 "10u" V 8300 2050 50  0000 R CNN
 F 2 "Capacitor_SMD:C_0805_2012Metric_Pad1.15x1.40mm_HandSolder" H 8238 1950 50  0001 C CNN
@@
 AR Path="/5EE5BDE4/5F11C2AA/5DB37044" Ref="C?"  Part="1"
 AR Path="/5F11EDFC/5DB37044" Ref="C93"  Part="1"
-F 0 "C51" V 8300 2650 50  0000 L CNN
+F 0 "C93" V 8300 2650 50  0000 L CNN
 F 1 "10u" V 8300 2550 50  0000 R CNN
 F 2 "Capacitor_SMD:C_0805_2012Metric_Pad1.15x1.40mm_HandSolder" H 8238 2450 50  0001 C CNN
@@
 AR Path="/5EE5BDE4/5F11C2AA/5DB4EB12" Ref="C?"  Part="1"
 AR Path="/5F11EDFC/5DB4EB12" Ref="C96"  Part="1"
-F 0 "C54" V 8800 2150 50  0000 L CNN
+F 0 "C96" V 8800 2150 50  0000 L CNN
 F 1 "10u" V 8800 2050 50  0000 R CNN
 F 2 "Capacitor_SMD:C_0805_2012Metric_Pad1.15x1.40mm_HandSolder" H 8738 1950 50  0001 C CNN
@@
 AR Path="/5EE5BDE4/5F11C2AA/5DB596AD" Ref="C?"  Part="1"
 AR Path="/5F11EDFC/5DB596AD" Ref="C97"  Part="1"
-F 0 "C55" V 8800 2650 50  0000 L CNN
+F 0 "C97" V 8800 2650 50  0000 L CNN
 F 1 "10u" V 8800 2550 50  0000 R CNN
 F 2 "Capacitor_SMD:C_0805_2012Metric_Pad1.15x1.40mm_HandSolder" H 8738 2450 50  0001 C CNN
@@
 AR Path="/5EE5BDE4/5F11C2AA/5DB7BE8B" Ref="C?"  Part="1"
 AR Path="/5F11EDFC/5DB7BE8B" Ref="C100"  Part="1"
-F 0 "C58" V 9300 2150 50  0000 L CNN
+F 0 "C100" V 9300 2150 50  0000 L CNN
 F 1 "10u" V 9300 2050 50  0000 R CNN
 F 2 "Capacitor_SMD:C_0805_2012Metric_Pad1.15x1.40mm_HandSolder" H 9238 1950 50  0001 C CNN
@@
 AR Path="/5EE5BDE4/5F11C2AA/5DB7BEA1" Ref="C?"  Part="1"
 AR Path="/5F11EDFC/5DB7BEA1" Ref="C101"  Part="1"
-F 0 "C59" V 9300 2650 50  0000 L CNN
+F 0 "C101" V 9300 2650 50  0000 L CNN
 F 1 "10u" V 9300 2550 50  0000 R CNN
 F 2 "Capacitor_SMD:C_0805_2012Metric_Pad1.15x1.40mm_HandSolder" H 9238 2450 50  0001 C CNN
@@
 AR Path="/5EE5BDE4/5F11C2AA/5EBF2A39" Ref="U?"  Part="1"
 AR Path="/5F11EDFC/5EBF2A39" Ref="U17"  Part="1"
-F 0 "U9" V 5304 2570 50  0000 R CNN
+F 0 "U17" V 5304 2570 50  0000 R CNN
 F 1 "AD8676xR" V 5395 2570 50  0000 R CNN
 F 2 "Package_SO:SOIC-8_3.9x4.9mm_P1.27mm" H 5450 2800 50  0001 C CNN
@@
 AR Path="/5EE5BDE4/5F11C2AA/5EBF3E04" Ref="U?"  Part="3"
 AR Path="/5F11EDFC/5EBF3E04" Ref="U17"  Part="3"
-F 0 "U9" H 9858 2396 50  0000 L CNN
+F 0 "U17" H 9858 2396 50  0000 L CNN
 F 1 "AD8676xR" H 9858 2305 50  0000 L CNN
 F 2 "Package_SO:SOIC-8_3.9x4.9mm_P1.27mm" H 9900 2350 50  0001 C CNN
@@
 AR Path="/5EE5BDE4/5F11C2AA/5EC22718" Ref="U?"  Part="1"
 AR Path="/5F11EDFC/5EC22718" Ref="U18"  Part="1"
-F 0 "U10" H 6800 3600 50  0000 L CNN
+F 0 "U18" H 6800 3600 50  0000 L CNN
 F 1 "AD8675" H 6750 3500 50  0000 L CNN
 F 2 "Package_SO:SOIC-8_3.9x4.9mm_P1.27mm" H 6950 4000 50  0001 C CNN
@@
 AR Path="/5EE5BDE4/5F11C2AA/5EE92855" Ref="C?"  Part="1"
 AR Path="/5F11EDFC/5EE92855" Ref="C95"  Part="1"
-F 0 "C26" V 8550 2650 50  0000 L CNN
+F 0 "C95" V 8550 2650 50  0000 L CNN
 F 1 "100n" V 8550 2550 50  0000 R CNN
 F 2 "Capacitor_SMD:C_0603_1608Metric_Pad1.05x0.95mm_HandSolder" H 8488 2450 50  0001 C CNN
@@
 AR Path="/5EE5BDE4/5F11C2AA/5EE92AC5" Ref="C?"  Part="1"
 AR Path="/5F11EDFC/5EE92AC5" Ref="C99"  Part="1"
-F 0 "C29" V 9050 2650 50  0000 L CNN
+F 0 "C99" V 9050 2650 50  0000 L CNN
 F 1 "100n" V 9050 2550 50  0000 R CNN
 F 2 "Capacitor_SMD:C_0603_1608Metric_Pad1.05x0.95mm_HandSolder" H 8988 2450 50  0001 C CNN
@@
 AR Path="/5EE5BDE4/5F11C2AA/5EE92D85" Ref="C?"  Part="1"
 AR Path="/5F11EDFC/5EE92D85" Ref="C98"  Part="1"
-F 0 "C27" V 9050 2150 50  0000 L CNN
+F 0 "C98" V 9050 2150 50  0000 L CNN
 F 1 "100n" V 9050 2050 50  0000 R CNN
 F 2 "Capacitor_SMD:C_0603_1608Metric_Pad1.05x0.95mm_HandSolder" H 8988 1950 50  0001 C CNN
@@
 AR Path="/5EE5BDE4/5F11C2AA/5EE931CA" Ref="C?"  Part="1"
 AR Path="/5F11EDFC/5EE931CA" Ref="C103"  Part="1"
-F 0 "C30" V 9550 2150 50  0000 L CNN
+F 0 "C103" V 9550 2150 50  0000 L CNN
 F 1 "100n" V 9550 2050 50  0000 R CNN
 F 2 "Capacitor_SMD:C_0603_1608Metric_Pad1.05x0.95mm_HandSolder" H 9488 1950 50  0001 C CNN
@@
 AR Path="/5EE5BDE4/5F11C2AA/5EE9354C" Ref="C?"  Part="1"
 AR Path="/5F11EDFC/5EE9354C" Ref="C104"  Part="1"
-F 0 "C31" V 9550 2650 50  0000 L CNN
+F 0 "C104" V 9550 2650 50  0000 L CNN
 F 1 "100n" V 9550 2550 50  0000 R CNN
 F 2 "Capacitor_SMD:C_0603_1608Metric_Pad1.05x0.95mm_HandSolder" H 9488 2450 50  0001 C CNN
@@
 AR Path="/5EE5BDE4/5F11C2AA/5EE955F2" Ref="C?"  Part="1"
 AR Path="/5F11EDFC/5EE955F2" Ref="C105"  Part="1"
-F 0 "C32" V 9700 4150 50  0000 L CNN
+F 0 "C105" V 9700 4150 50  0000 L CNN
 F 1 "100n" V 9700 4050 50  0000 R CNN
 F 2 "Capacitor_SMD:C_0603_1608Metric_Pad1.05x0.95mm_HandSolder" H 9638 3950 50  0001 C CNN
@@
 AR Path="/5EE5BDE4/5F11C2AA/5ED378D9" Ref="C?"  Part="1"
 AR Path="/5F11EDFC/5ED378D9" Ref="C89"  Part="1"
-F 0 "C71" H 4915 2346 50  0000 L CNN
+F 0 "C89" H 4915 2346 50  0000 L CNN
 F 1 "10p" H 4915 2255 50  0000 L CNN
 F 2 "Capacitor_SMD:C_0603_1608Metric_Pad1.05x0.95mm_HandSolder" H 4838 2150 50  0001 C CNN
@@
 AR Path="/5EE5BDE4/5F11C2AA/5ED4490E" Ref="C?"  Part="1"
 AR Path="/5F11EDFC/5ED4490E" Ref="C90"  Part="1"
-F 0 "C72" H 4915 5196 50  0000 L CNN
+F 0 "C90" H 4915 5196 50  0000 L CNN
 F 1 "10p" H 4915 5105 50  0000 L CNN
 F 2 "Capacitor_SMD:C_0603_1608Metric_Pad1.05x0.95mm_HandSolder" H 4838 5000 50  0001 C CNN
@@
 AR Path="/5EE5BDE4/5F11C2AA/5EBF327E" Ref="U?"  Part="2"
 AR Path="/5F11EDFC/5EBF327E" Ref="U17"  Part="2"
-F 0 "U9" V 5396 4370 50  0000 R CNN
+F 0 "U17" V 5396 4370 50  0000 R CNN
 F 1 "AD8676xR" V 5305 4370 50  0000 R CNN
 F 2 "Package_SO:SOIC-8_3.9x4.9mm_P1.27mm" H 5450 4600 50  0001 C CNN
@@
 AR Path="/5EE5BDE4/5F11C2AA/5F0961D2" Ref="JP?"  Part="1"
 AR Path="/5F11EDFC/5F0961D2" Ref="JP10"  Part="1"
-F 0 "JP5" H 7700 3923 50  0000 C CNN
+F 0 "JP10" H 7700 3923 50  0000 C CNN
 F 1 "Jumper" H 7700 3923 50  0001 C CNN
 F 2 "Connector_PinHeader_2.54mm:PinHeader_1x02_P2.54mm_Vertical" H 7700 3750 50  0001 C CNN

Commit message: Layout progress
Changed lines of the file:
@@
 AR Path="/5EE5BDE4/5F11C2AA/5DA35D26" Ref="U?"  Part="1"
 AR Path="/5F11EDFC/5DA35D26" Ref="U16"  Part="1"
-F 0 "U16" H 5100 3850 50  0000 L CNN
+F 0 "U8" H 5100 3850 50  0000 L CNN
 F 1 "AD5781" H 5000 3750 50  0000 L CNN
 F 2 "Package_SO:TSSOP-20_4.4x6.5mm_P0.65mm" H 4550 3800 50  0001 C CNN
@@
 AR Path="/5EE5BDE4/5F11C2AA/5DA6205A" Ref="C?"  Part="1"
 AR Path="/5F11EDFC/5DA6205A" Ref="C91"  Part="1"
-F 0 "C91" H 6315 3546 50  0000 L CNN
+F 0 "C28" H 6315 3546 50  0000 L CNN
 F 1 "10p" H 6315 3455 50  0000 L CNN
 F 2 "Capacitor_SMD:C_0603_1608Metric_Pad1.05x0.95mm_HandSolder" H 6238 3350 50  0001 C CNN
@@
 AR Path="/5EE5BDE4/5F11C2AA/5DAF59CE" Ref="C?"  Part="1"
 AR Path="/5F11EDFC/5DAF59CE" Ref="C102"  Part="1"
-F 0 "C102" V 9450 4150 50  0000 L CNN
+F 0 "C47" V 9450 4150 50  0000 L CNN
 F 1 "10u" V 9450 4050 50  0000 R CNN
 F 2 "Capacitor_SMD:C_0805_2012Metric_Pad1.15x1.40mm_HandSolder" H 9388 3950 50  0001 C CNN
@@
 AR Path="/5EE5BDE4/5F11C2AA/5DAFF8A7" Ref="C?"  Part="1"
 AR Path="/5F11EDFC/5DAFF8A7" Ref="C94"  Part="1"
-F 0 "C94" V 8550 2150 50  0000 L CNN
+F 0 "C52" V 8550 2150 50  0000 L CNN
 F 1 "100n" V 8550 2050 50  0000 R CNN
 F 2 "Capacitor_SMD:C_0603_1608Metric_Pad1.05x0.95mm_HandSolder" H 8488 1950 50  0001 C CNN
@@
 AR Path="/5EE5BDE4/5F11C2AA/5DAFF8B1" Ref="C?"  Part="1"
 AR Path="/5F11EDFC/5DAFF8B1" Ref="C92"  Part="1"
-F 0 "C92" V 8300 2150 50  0000 L CNN
+F 0 "C50" V 8300 2150 50  0000 L CNN
 F 1 "10u" V 8300 2050 50  0000 R CNN
 F 2 "Capacitor_SMD:C_0805_2012Metric_Pad1.15x1.40mm_HandSolder" H 8238 1950 50  0001 C CNN
@@
 AR Path="/5EE5BDE4/5F11C2AA/5DB37044" Ref="C?"  Part="1"
 AR Path="/5F11EDFC/5DB37044" Ref="C93"  Part="1"
-F 0 "C93" V 8300 2650 50  0000 L CNN
+F 0 "C51" V 8300 2650 50  0000 L CNN
 F 1 "10u" V 8300 2550 50  0000 R CNN
 F 2 "Capacitor_SMD:C_0805_2012Metric_Pad1.15x1.40mm_HandSolder" H 8238 2450 50  0001 C CNN
@@
 AR Path="/5EE5BDE4/5F11C2AA/5DB4EB12" Ref="C?"  Part="1"
 AR Path="/5F11EDFC/5DB4EB12" Ref="C96"  Part="1"
-F 0 "C96" V 8800 2150 50  0000 L CNN
+F 0 "C54" V 8800 2150 50  0000 L CNN
 F 1 "10u" V 8800 2050 50  0000 R CNN
 F 2 "Capacitor_SMD:C_0805_2012Metric_Pad1.15x1.40mm_HandSolder" H 8738 1950 50  0001 C CNN
@@
 AR Path="/5EE5BDE4/5F11C2AA/5DB596AD" Ref="C?"  Part="1"
 AR Path="/5F11EDFC/5DB596AD" Ref="C97"  Part="1"
-F 0 "C97" V 8800 2650 50  0000 L CNN
+F 0 "C55" V 8800 2650 50  0000 L CNN
 F 1 "10u" V 8800 2550 50  0000 R CNN
 F 2 "Capacitor_SMD:C_0805_2012Metric_Pad1.15x1.40mm_HandSolder" H 8738 2450 50  0001 C CNN
@@
 AR Path="/5EE5BDE4/5F11C2AA/5DB7BE8B" Ref="C?"  Part="1"
 AR Path="/5F11EDFC/5DB7BE8B" Ref="C100"  Part="1"
-F 0 "C100" V 9300 2150 50  0000 L CNN
+F 0 "C58" V 9300 2150 50  0000 L CNN
 F 1 "10u" V 9300 2050 50  0000 R CNN
 F 2 "Capacitor_SMD:C_0805_2012Metric_Pad1.15x1.40mm_HandSolder" H 9238 1950 50  0001 C CNN
@@
 AR Path="/5EE5BDE4/5F11C2AA/5DB7BEA1" Ref="C?"  Part="1"
 AR Path="/5F11EDFC/5DB7BEA1" Ref="C101"  Part="1"
-F 0 "C101" V 9300 2650 50  0000 L CNN
+F 0 "C59" V 9300 2650 50  0000 L CNN
 F 1 "10u" V 9300 2550 50  0000 R CNN
 F 2 "Capacitor_SMD:C_0805_2012Metric_Pad1.15x1.40mm_HandSolder" H 9238 2450 50  0001 C CNN
@@
 AR Path="/5EE5BDE4/5F11C2AA/5EBF2A39" Ref="U?"  Part="1"
 AR Path="/5F11EDFC/5EBF2A39" Ref="U17"  Part="1"
-F 0 "U17" V 5304 2570 50  0000 R CNN
+F 0 "U9" V 5304 2570 50  0000 R CNN
 F 1 "AD8676xR" V 5395 2570 50  0000 R CNN
 F 2 "Package_SO:SOIC-8_3.9x4.9mm_P1.27mm" H 5450 2800 50  0001 C CNN
@@
 AR Path="/5EE5BDE4/5F11C2AA/5EBF3E04" Ref="U?"  Part="3"
 AR Path="/5F11EDFC/5EBF3E04" Ref="U17"  Part="3"
-F 0 "U17" H 9858 2396 50  0000 L CNN
+F 0 "U9" H 9858 2396 50  0000 L CNN
 F 1 "AD8676xR" H 9858 2305 50  0000 L CNN
 F 2 "Package_SO:SOIC-8_3.9x4.9mm_P1.27mm" H 9900 2350 50  0001 C CNN
@@
 AR Path="/5EE5BDE4/5F11C2AA/5EC22718" Ref="U?"  Part="1"
 AR Path="/5F11EDFC/5EC22718" Ref="U18"  Part="1"
-F 0 "U18" H 6800 3600 50  0000 L CNN
+F 0 "U10" H 6800 3600 50  0000 L CNN
 F 1 "AD8675" H 6750 3500 50  0000 L CNN
 F 2 "Package_SO:SOIC-8_3.9x4.9mm_P1.27mm" H 6950 4000 50  0001 C CNN
@@
 AR Path="/5EE5BDE4/5F11C2AA/5EE92855" Ref="C?"  Part="1"
 AR Path="/5F11EDFC/5EE92855" Ref="C95"  Part="1"
-F 0 "C95" V 8550 2650 50  0000 L CNN
+F 0 "C26" V 8550 2650 50  0000 L CNN
 F 1 "100n" V 8550 2550 50  0000 R CNN
 F 2 "Capacitor_SMD:C_0603_1608Metric_Pad1.05x0.95mm_HandSolder" H 8488 2450 50  0001 C CNN
@@
 AR Path="/5EE5BDE4/5F11C2AA/5EE92AC5" Ref="C?"  Part="1"
 AR Path="/5F11EDFC/5EE92AC5" Ref="C99"  Part="1"
-F 0 "C99" V 9050 2650 50  0000 L CNN
+F 0 "C29" V 9050 2650 50  0000 L CNN
 F 1 "100n" V 9050 2550 50  0000 R CNN
 F 2 "Capacitor_SMD:C_0603_1608Metric_Pad1.05x0.95mm_HandSolder" H 8988 2450 50  0001 C CNN
@@
 AR Path="/5EE5BDE4/5F11C2AA/5EE92D85" Ref="C?"  Part="1"
 AR Path="/5F11EDFC/5EE92D85" Ref="C98"  Part="1"
-F 0 "C98" V 9050 2150 50  0000 L CNN
+F 0 "C27" V 9050 2150 50  0000 L CNN
 F 1 "100n" V 9050 2050 50  0000 R CNN
 F 2 "Capacitor_SMD:C_0603_1608Metric_Pad1.05x0.95mm_HandSolder" H 8988 1950 50  0001 C CNN
@@
 AR Path="/5EE5BDE4/5F11C2AA/5EE931CA" Ref="C?"  Part="1"
 AR Path="/5F11EDFC/5EE931CA" Ref="C103"  Part="1"
-F 0 "C103" V 9550 2150 50  0000 L CNN
+F 0 "C30" V 9550 2150 50  0000 L CNN
 F 1 "100n" V 9550 2050 50  0000 R CNN
 F 2 "Capacitor_SMD:C_0603_1608Metric_Pad1.05x0.95mm_HandSolder" H 9488 1950 50  0001 C CNN
@@
 AR Path="/5EE5BDE4/5F11C2AA/5EE9354C" Ref="C?"  Part="1"
 AR Path="/5F11EDFC/5EE9354C" Ref="C104"  Part="1"
-F 0 "C104" V 9550 2650 50  0000 L CNN
+F 0 "C31" V 9550 2650 50  0000 L CNN
 F 1 "100n" V 9550 2550 50  0000 R CNN
 F 2 "Capacitor_SMD:C_0603_1608Metric_Pad1.05x0.95mm_HandSolder" H 9488 2450 50  0001 C CNN
@@
 AR Path="/5EE5BDE4/5F11C2AA/5EE955F2" Ref="C?"  Part="1"
 AR Path="/5F11EDFC/5EE955F2" Ref="C105"  Part="1"
-F 0 "C105" V 9700 4150 50  0000 L CNN
+F 0 "C32" V 9700 4150 50  0000 L CNN
 F 1 "100n" V 9700 4050 50  0000 R CNN
 F 2 "Capacitor_SMD:C_0603_1608Metric_Pad1.05x0.95mm_HandSolder" H 9638 3950 50  0001 C CNN
@@
 AR Path="/5EE5BDE4/5F11C2AA/5ED378D9" Ref="C?"  Part="1"
 AR Path="/5F11EDFC/5ED378D9" Ref="C89"  Part="1"
-F 0 "C89" H 4915 2346 50  0000 L CNN
+F 0 "C71" H 4915 2346 50  0000 L CNN
 F 1 "10p" H 4915 2255 50  0000 L CNN
 F 2 "Capacitor_SMD:C_0603_1608Metric_Pad1.05x0.95mm_HandSolder" H 4838 2150 50  0001 C CNN
@@
 AR Path="/5EE5BDE4/5F11C2AA/5ED4490E" Ref="C?"  Part="1"
 AR Path="/5F11EDFC/5ED4490E" Ref="C90"  Part="1"
-F 0 "C90" H 4915 5196 50  0000 L CNN
+F 0 "C72" H 4915 5196 50  0000 L CNN
 F 1 "10p" H 4915 5105 50  0000 L CNN
 F 2 "Capacitor_SMD:C_0603_1608Metric_Pad1.05x0.95mm_HandSolder" H 4838 5000 50  0001 C CNN
@@
 AR Path="/5EE5BDE4/5F11C2AA/5EBF327E" Ref="U?"  Part="2"
 AR Path="/5F11EDFC/5EBF327E" Ref="U17"  Part="2"
-F 0 "U17" V 5396 4370 50  0000 R CNN
+F 0 "U9" V 5396 4370 50  0000 R CNN
 F 1 "AD8676xR" V 5305 4370 50  0000 R CNN
 F 2 "Package_SO:SOIC-8_3.9x4.9mm_P1.27mm" H 5450 4600 50  0001 C CNN
@@
 AR Path="/5EE5BDE4/5F11C2AA/5F0961D2" Ref="JP?"  Part="1"
 AR Path="/5F11EDFC/5F0961D2" Ref="JP10"  Part="1"
-F 0 "JP10" H 7700 3923 50  0000 C CNN
+F 0 "JP5" H 7700 3923 50  0000 C CNN
 F 1 "Jumper" H 7700 3923 50  0001 C CNN
 F 2 "Connector_PinHeader_2.54mm:PinHeader_1x02_P2.54mm_Vertical" H 7700 3750 50  0001 C CNN
