File: Electronics/Supply-Board/Supply-Board.kicad_pcb (KiCad board)
At the start: 2 copper layers, 160 x 99.5 mm, 91 parts, among them J1 DB25_Female_MountingHoles, J2 PE, J3 L, J4 N, T1 Transformer_1P_2S, T2 Transformer_1P_2S, U1 LM317, U2 LM337, U3 240R, U4 LM337, U5 traco_TSR_0.5-2433, U6 LM75C

Commit message: Fixed values in schematic
Parts:
- C1, C2, C3, C4: value 1000u -> 1500u
- C13, C14, C15, C16: value 1000u -> 820u
- C17, C18, C5, C6: value 100n -> 470n
- C20, C24, C25, C26: value 10u -> 4u7
- D1, D4: value VC 5,0/2/15 -> B250S2A
- R10, R4: value 120R -> 240R
- R15, R16: value 10k -> 2k7
- R2: value 1k3 -> 2k6
- R8: value 1k8 -> 3k6
- T1: value Transformer_1P_2S -> VC 5,0/2/15
- T2: value Transformer_1P_2S -> VC 5,0/2/18
- U3: value 240R -> LM317
- renumbered REF** to e
